Commit message: Explored cone detection with depth camera, and implemented gps localisation

File: src/avone/description/depthcamera.xacro (robot description, xacro)
@@ -27,4 +27,5 @@
             <visualize>true</visualize>
             <update_rate>10</update_rate>
+            <topic>depth/image_raw</topic>
             <camera>
                 <horizontal_fov>1.089</horizontal_fov>
@@ -39,9 +40,4 @@
                 </clip>
             </camera>
-            <plugin name="depthcamera_controller" filename="libgazebo_ros_depthcamera.so">
-                <frame_name>depthcamera_link_optical</frame_name>
-                <min_depth>0.1</min_depth>
-                <max_depth>100.0</max_depth>
-            </plugin>
         </sensor>
     </gazebo>

File: src/avone/description/rgbdcamera.xacro (robot description, xacro)
@@ -1,51 +1,39 @@
 <?xml version="1.0"?>
-<robot xmlns:xacro="http://www.ros.org/wiki/xacro" >
-    <joint name="rgbdcamera_joint" type="fixed">
-        <parent link="chassis"/>
-        <child link="rgbdcamera_link"/>
-        <origin xyz="0.6909 0 0.772413" rpy="0 0 0"/>
-    </joint>
-    <link name="rgbdcamera_link">
-        <visual>
-            <geometry>
-                <box size="0.010 0.03 0.03"/>
-            </geometry>
-            <material name="red"/>
-        </visual>
-    </link>
-    <joint name="rgbdcamera_optical_joint" type="fixed">
-        <parent link="rgbdcamera_link"/>
-        <child link="rgbdcamera_link_optical"/>
-        <origin xyz="0 0 0" rpy="0 0 0"/>
-    </joint>
-    <link name="rgbdcamera_link_optical"></link>
-    <gazebo reference="rgbdcamera_link">
-        <material>Gazebo/Red</material>
-        <sensor name="rgbdcamera" type="rgbd">
-            <gz_frame_id>rgbdcamera_link_optical</gz_frame_id>
-            <pose> 0 0 0 0 0 0 </pose>
-            <visualize>true</visualize>
-            <update_rate>10</update_rate>
-             <topic>rgbdcamera</topic>
-            <camera>
-                <horizontal_fov>1.1</horizontal_fov>
-                <image>
-                    <format>R8G8B8</format>
-                    <width>1920</width>
-                    <height>1080</height>
-                </image>
-                <clip>
-                    <near>0.05</near>
-                    <far>50.0</far>
-                </clip>
-            </camera>
-            <!--
-            <plugin name="camera_controller" filename="libgazebo_ros_camera.so">
-                <frame_name>rgbdcamera_link_optical</frame_name>
-                <min_depth>0.1</min_depth>
-                <max_depth>100.0</max_depth>
-            </plugin>
-            -->
-        </sensor>
-    </gazebo>
+<robot xmlns:xacro="http://www.ros.org/wiki/xacro">
+  <!-- 1) raw camera on the chassis -->
+  <joint name="rgbdcamera_joint" type="fixed">
+    <parent link="chassis"/>
+    <child  link="rgbdcamera_link"/>
+    <origin xyz="0.6909 0 0.772413" rpy="0 0 0"/>
+  </joint>
+  <link name="rgbdcamera_link"/>
+  <!-- 2) optical frame, with X→right, Y→down, Z→forward -->
+  <joint name="rgbdcamera_optical_joint" type="fixed">
+    <parent link="rgbdcamera_link"/>
+    <child  link="rgbdcamera_link_optical"/>
+    <!-- roll = -90°, pitch = 0, yaw = -90° -->
+    <origin xyz="0 0 0" rpy="0 0 0"/>
+  </joint>
+  <link name="rgbdcamera_link_optical"/>
+  <!-- 3) Gazebo ROS2 camera plugin on the OPTICAL link -->
+  <gazebo reference="rgbdcamera_link_optical">
+    <sensor name="rgbdcamera" type="rgbd">
+      <topic>rgbdcamera</topic>
+      <gz_frame_id>rgbdcamera_link</gz_frame_id>
+      <pose>0 0 0 0 0 0</pose>
+      <update_rate>30</update_rate>
+      <camera>
+        <horizontal_fov>1.91986</horizontal_fov>
+        <image>
+          <format>R8G8B8</format>
+          <width>1280</width>
+          <height>720</height>
+        </image>
+        <clip>
+          <near>0.3</near>
+          <far>20.0</far>
+        </clip>
+      </camera>
+    </sensor>
+  </gazebo>
 </robot>

File: src/avone/description/robot.urdf.xacro (robot description, xacro)
@@ -4,8 +4,8 @@
     <xacro:include filename="ros2_control.xacro" />
     <xacro:include filename="gazebo_control.xacro"/>
-    <xacro:include filename="camera.xacro" />
-    <!--<xacro:include filename="depthcamera.xacro" /> -->
-  <!-- <xacro:include filename="rgbdcamera.xacro" /> -->
+    <!-- <xacro:include filename="camera.xacro" />  -->
+    <!-- <xacro:include filename="depthcamera.xacro" /> -->
+   <xacro:include filename="rgbdcamera.xacro" />
    <xacro:include filename="sensors.xacro" />
-   <xacro:include filename="lidar.xacro" />
+   <!-- <xacro:include filename="lidar.xacro" />  -->
 </robot>

File: src/avone/description/sensors.xacro (robot description, xacro)
@@ -4,17 +4,69 @@
         <parent link="chassis"/>
         <child link="imu_link"/>
-        <origin xyz="0 0 0.3" rpy="0 0 0"/>  <!-- e.g. 5 cm above chassis CG -->
+          <origin xyz="0.5 0 0.5" rpy="0 0 0"/>
     </joint>
-   <link name="imu_link">
-  <!-- no <sensor> here! -->
-</link>
-<gazebo reference="imu_link">
-   <sensor name="imu_sensor" type="imu">
-    <gz_frame_id>imu_link</gz_frame_id>
-                    <always_on>1</always_on>
-                    <update_rate>10</update_rate>
-                    <visualize>true</visualize>
-                    <topic>imu</topic>
-                </sensor>
-</gazebo>
+  <link name="imu_link"></link>
+  <gazebo reference="imu_link">
+    <sensor name="imu_sensor" type="imu">
+      <gz_frame_id>imu_link</gz_frame_id>
+      <always_on>1</always_on>
+      <update_rate>50</update_rate>
+      <visualize>true</visualize>
+      <topic>imu</topic>
+    </sensor>
+  </gazebo>
+  <!-- FRONT GPS ANTENNA -->
+  <joint name="gps_antenna1_joint" type="fixed">
+        <parent link="chassis"/>
+        <child link="gps_antenna1_link"/>
+          <origin xyz="2.3674 0 0.2977" rpy="0 0 0"/>
+    </joint>
+  <link name="gps_antenna1_link">
+    <visual>
+      <geometry>
+        <cylinder radius="0.0625" length="0.085"/>
+      </geometry>
+      <material name="white"/>
+    </visual>
+    <collision>
+      <geometry>
+        <cylinder radius="0.0625" length="0.085"/>
+      </geometry>
+    </collision>
+  </link>
+  <gazebo reference="gps_antenna1_link">
+    <sensor name="navsat1" type="navsat">
+    <gz_frame_id>gps_antenna1_link</gz_frame_id>
+      <always_on>1</always_on>
+      <update_rate>50</update_rate>
+      <topic>navsat1</topic>
+    </sensor>
+  </gazebo>
+  <!-- REAR GPS ANTENNA -->
+<joint name="gps_antenna2_joint" type="fixed">
+        <parent link="chassis"/>
+        <child link="gps_antenna2_link"/>
+          <origin xyz="0.2299 0 0.4025" rpy="0 0 0"/>
+    </joint>
+  <link name="gps_antenna2_link">
+    <visual>
+      <geometry>
+        <cylinder radius="0.0625" length="0.085"/>
+      </geometry>
+      <material name="white"/>
+    </visual>
+    <collision>
+      <geometry>
+        <cylinder radius="0.0625" length="0.085"/>
+      </geometry>
+    </collision>
+  </link>
+  <gazebo reference="gps_antenna2_link">
+    <sensor name="navsat2" type="navsat">
+    <gz_frame_id>gps_antenna2_link</gz_frame_id>
+      <always_on>1</always_on>
+      <update_rate>50</update_rate>
+      <topic>navsat2</topic>
+    </sensor>
+  </gazebo>
 </robot>
