Commit message: push before test on NUC, better NAV2, and R2D

File: src/avone/description/lidar.xacro (robot description, xacro)
@@ -4,5 +4,5 @@
         <parent link="chassis"/>
         <child link="laser_frame"/>
-         <origin xyz="2.3674 0 0.2977" rpy="0 0 0"/>
+         <origin xyz="2.244 0 0.3464" rpy="0 0 0"/>
         <!-- <origin xyz="0.6909 0 0.772413" rpy="0 0.4 0"/> -->
     </joint>

File: src/avone/description/robot.urdf.xacro (robot description, xacro)
@@ -1,21 +1,8 @@
 <?xml version="1.0"?>
 <robot xmlns:xacro="http://www.ros.org/wiki/xacro" name="robot">
-  <!-- 1) Declare your flags -->
-  <!-- <xacro:arg name="use_sim"       default="true"/>
-  <xacro:arg name="can_interface" default="vcan0"/>
-  <xacro:arg name="steer_node_id" default="2"/>
-  <xacro:arg name="motor_node_id" default="1"/>  -->
   <!-- 2) Core links/visuals etc -->
   <xacro:include filename="robot_core.xacro"/>
-  <!-- 3) Simulation ros2_control -->
-  <!-- <xacro:if value="$(arg use_sim)"> -->
-    <xacro:include filename="ros2_control.xacro"/>
-    <!-- if you want gazebo_control in sim, uncomment this too -->
-    <!-- <xacro:include filename="gazebo_control.xacro"/> -->
-  <!-- </xacro:if> -->
-  <!-- 4) Real-hardware ros2_control -->
-  <!-- <xacro:unless value="$(arg use_sim)"> -->
-    <!-- <xacro:include filename="ros2_control_hardware.xacro"/> -->
-  <!-- </xacro:unless> -->
+  <!-- <xacro:include filename="ros2_control.xacro"/> -->
+  <xacro:include filename="ros2_control_hardware.xacro"/>
   <!-- 5) Sensors, cameras, lidar, etc. -->
   <xacro:include filename="camera.xacro"/>

File: src/avone/description/ros2_control_hardware.xacro (robot description, xacro)
@@ -4,4 +4,5 @@
     <hardware>
       <plugin>avone/AvoneSystemHardware</plugin>
+      <!-- Your existing params -->
       <param name="max_steer_angle">1.3</param>
       <param name="min_steer_angle">-1.3</param>
@@ -11,5 +12,4 @@
       <param name="read_timeout_ms">20</param>
       <param name="l_motor_can_id">0x8CF11E05</param>
-      <!-- set right as same as left until figure out motor controller  -->
       <param name="r_motor_can_id">0x8CF11E06</param>
       <param name="steer_can_id">0x006</param>
@@ -17,32 +17,50 @@
       <param name="cmd_r_motor_can_id">0x0C</param>
       <param name="cmd_steer_can_id">0x004</param>
+      <!-- NEW: safety/watchdog controls -->
+      <!-- Which feedback signals are required before arming & during run -->
+      <param name="require_rlmotor">false</param>
+      <param name="require_rrmotor">false</param>
+      <param name="require_steer">false</param>
+      <!-- Activation: wait up to this long for first feedback frames -->
+      <param name="startup_validation_ms">800</param>
+      <!-- Runtime: max allowed age for any required signal -->
+      <param name="link_loss_timeout_ms">250</param>
+            <!-- LiDAR watchdog -->
+      <param name="require_lidar">false</param>
+      <param name="lidar_topic">/lidar</param>
+      <!-- Choose the actual ROS 2 type your stack publishes: -->
+      <param name="lidar_ros_type">sensor_msgs/msg/PointCloud2</param>
+      <!-- or -->
+      <!-- <param name="lidar_ros_type">sensor_msgs/msg/LaserScan</param> -->
+      <param name="lidar_timeout_ms">300</param>
+      <!-- Ready-To-Drive signalling -->
+      <param name="r2d_topic">/ready_to_drive</param>
+      <param name="r2d_can_heartbeat">true</param>
+      <param name="r2d_can_id">0x110</param>
+      <param name="r2d_can_period_ms">50</param>
     </hardware>
-  <!-- front steering -->
-  <joint name="LSteer">
-    <command_interface name="position"/>
-    <state_interface   name="position"/>
-  </joint>
-  <joint name="RSteer">
-    <command_interface name="position"/>
-    <state_interface   name="position"/>
-  </joint>
-  <!-- rear drive -->
-  <joint name="RLMotor">
-    <command_interface name="velocity"/>
-    <state_interface   name="velocity"/>
-    <state_interface   name="position"/>
-  </joint>
-  <joint name="RRMotor">
-    <command_interface name="velocity"/>
-    <state_interface   name="velocity"/>
-    <state_interface   name="position"/>
-  </joint>
-  <!-- Front wheels just mirroring rear -->
-  <joint name="FLWheel">
-    <state_interface   name="position"/>
-  </joint>
-  <joint name="FRWheel">
-    <state_interface   name="position"/>
-  </joint>
-</ros2_control>
+    <!-- front steering -->
+    <joint name="LSteer">
+      <command_interface name="position"/>
+      <state_interface   name="position"/>
+    </joint>
+    <joint name="RSteer">
+      <command_interface name="position"/>
+      <state_interface   name="position"/>
+    </joint>
+    <!-- rear drive -->
+    <joint name="RLMotor">
+      <command_interface name="velocity"/>
+      <state_interface   name="velocity"/>
+      <state_interface   name="position"/>
+    </joint>
+    <joint name="RRMotor">
+      <command_interface name="velocity"/>
+      <state_interface   name="velocity"/>
+      <state_interface   name="position"/>
+    </joint>
+    <!-- front wheels (pos only) -->
+    <joint name="FLWheel"><state_interface name="position"/></joint>
+    <joint name="FRWheel"><state_interface name="position"/></joint>
+  </ros2_control>
 </robot>

File: src/avone/description/sensors.xacro (robot description, xacro)
@@ -4,5 +4,5 @@
         <parent link="chassis"/>
         <child link="imu_link"/>
-          <origin xyz="0.5 0 0.5" rpy="0 0 0"/>
+          <origin xyz="0.450 0 0.39137" rpy="0 0 0"/>
     </joint>
   <link name="imu_link"></link>
@@ -20,8 +20,8 @@
         <parent link="chassis"/>
         <child link="gps_antenna1_link"/>
-          <origin xyz="2.3674 0 0.2977" rpy="0 0 0"/>
+          <origin xyz="0.0312 0 0.3924" rpy="0 0 0"/>
     </joint>
   <link name="gps_antenna1_link">
-    <!-- <visual>
+    <visual>
       <geometry>
         <cylinder radius="0.0625" length="0.085"/>
@@ -33,5 +33,5 @@
         <cylinder radius="0.0625" length="0.085"/>
       </geometry>
-    </collision> -->
+    </collision>
   </link>
   <gazebo reference="gps_antenna1_link">
@@ -43,12 +43,11 @@
     </sensor>
   </gazebo>
-  <!-- REAR GPS ANTENNA -->
 <joint name="gps_antenna2_joint" type="fixed">
         <parent link="chassis"/>
         <child link="gps_antenna2_link"/>
-          <origin xyz="0.2299 0 0.4025" rpy="0 0 0"/>
+          <origin xyz="2.131 0 0.3924" rpy="0 0 0"/>
     </joint>
   <link name="gps_antenna2_link">
-    <!-- <visual>
+   <visual>
       <geometry>
         <cylinder radius="0.0625" length="0.085"/>
@@ -60,5 +59,5 @@
         <cylinder radius="0.0625" length="0.085"/>
       </geometry>
-    </collision> -->
+    </collision>
   </link>
   <gazebo reference="gps_antenna2_link">
