Commit message: Fixed odom reading through ekf, much more accurate

File: src/avone/description/robot_core.xacro (robot description, xacro)
@@ -146,6 +146,16 @@
         <child link="left_motor"/>
         <axis xyz="0 0 -1"/>
-     <dynamics damping="0.2" friction="0.1"/>
-      <limit effort="50" velocity="50"/>  <!-- up to 20 m/s -->    </joint>
+     <dynamics damping="0.1" friction="0.48"/>
+      <limit
+          effort="91.0"
+          velocity="100.7"/>
+        <!--
+            effort (Nm) = kT × I_cont
+              ≈ 0.955 Nm/A × 95 A = 91 Nm
+            velocity (rad/s) = Kv × V
+              ≈ (10 rpm/V × 96 V) × (2π/60) ≈ 100.7 rad/s
+            :contentReference[oaicite:0]{index=0}
+        -->
+      </joint>
     <link name="left_motor">
         <visual>
@@ -160,5 +170,6 @@
             <origin xyz="-8.09391e-17 7.65875e-18 0.17" rpy="1.5708 0 0"/>
             <geometry>
-                    <sphere radius="0.2"/>
+                     <!--<mesh filename="file:///home/jay/ros2_ws/src/avone/description/assets/wheel.stl"/>    -->
+                                        <sphere radius="0.203"/>
                  <!--  <box size="0.3 0.3 0.15"/> -->
             </geometry>
@@ -177,6 +188,9 @@
         <child link="right_motor"/>
         <axis xyz="0 0 1"/>
-      <dynamics damping="0.2" friction="0.1"/>
-      <limit effort="50" velocity="50"/>  <!-- up to 20 m/s -->    </joint>
+      <dynamics damping="0.1" friction="0.48"/>
+      <limit
+          effort="91.0"
+          velocity="100.7"/>
+    </joint>
     <link name="right_motor">
         <visual>
@@ -191,5 +205,5 @@
             <origin xyz="-1.59877e-17 7.65404e-18 0.17" rpy="1.5708 0 0"/>
             <geometry>
-                     <sphere radius="0.2"/>
+                     <sphere radius="0.203"/>
                  <!--  <box size="0.3 0.3 0.15"/> -->
             </geometry>
@@ -209,5 +223,5 @@
         <child link="front_right_wheel_hub"/>
         <axis xyz="0 0 -1"/>
-        <limit effort="100" velocity="20" lower="-0.8" upper="0.8"/>
+        <limit effort="100" velocity="20" lower="-0.4" upper="0.4"/>
           <dynamics damping="0.1" friction="0.05"/>
     </joint>
@@ -255,6 +269,6 @@
             <origin xyz="2.22045e-16 0 0.17" rpy="1.5708 0 1.5708"/>
             <geometry>
-                   <!-- <mesh filename="file:///home/jay/ros2_ws/src/avone/description/assets/wheel.stl"/>      -->
-                    <sphere radius="0.2"/>
+                   <!--<mesh filename="file:///home/jay/ros2_ws/src/avone/description/assets/wheel.stl"/>    -->
+                                        <sphere radius="0.203"/>
                  <!--  <box size="0.3 0.3 0.15"/> -->
             </geometry>
@@ -273,5 +287,5 @@
         <child link="front_left_wheel_hub"/>
         <axis xyz="0 0 -1"/>
-         <limit effort="100" velocity="20" lower="-0.8" upper="0.8"/>
+         <limit effort="100" velocity="20" lower="-0.4" upper="0.4"/>
           <dynamics damping="0.1" friction="0.05"/>
     </joint>
@@ -319,5 +333,6 @@
         <origin xyz="0 0 0.17" rpy="1.5708 0 0"/>
         <geometry>
-                     <sphere radius="0.2"/>
+                      <!--<mesh filename="file:///home/jay/ros2_ws/src/avone/description/assets/wheel.stl"/>    -->
+                                        <sphere radius="0.203"/>
                  <!--  <box size="0.3 0.3 0.15"/> -->
         </geometry>

File: src/avone/description/sensors.xacro (robot description, xacro)
@@ -4,5 +4,5 @@
         <parent link="chassis"/>
         <child link="imu_link"/>
-        <origin xyz="0.6909 0 0.772413" rpy="0 0 0"/>
+        <origin xyz="0 0 0.3" rpy="0 0 0"/>  <!-- e.g. 5 cm above chassis CG -->
     </joint>
    <link name="imu_link">

Commit message: final git push before re-organisation for hardware implementation

File: src/avone/description/robot_core.xacro (robot description, xacro)
@@ -22,5 +22,5 @@
         <parent link="base_link"/>
         <child link="base_footprint"/>
-        <origin xyz="0 0 0" rpy="0 0 0"/>
+        <origin xyz="1.0 0 0" rpy="0 0 0"/>
     </joint>
     <link name="base_footprint">

Commit message: updated until first connection between avone and nuc

File: src/avone/description/robot_core.xacro (robot description, xacro)
@@ -146,8 +146,9 @@
         <child link="left_motor"/>
         <axis xyz="0 0 -1"/>
-     <dynamics damping="0.1" friction="0.48"/>
+     <dynamics damping="0.02" friction="0.2"/>
       <limit
-          effort="91.0"
-          velocity="100.7"/>
+          effort="108.6"
+          velocity="36.65"/>
+          <!-- NEED TO FIND THIS ^^ -->
         <!--
             effort (Nm) = kT × I_cont
@@ -188,8 +189,8 @@
         <child link="right_motor"/>
         <axis xyz="0 0 1"/>
-      <dynamics damping="0.1" friction="0.48"/>
+      <dynamics damping="0.02" friction="0.2"/>
       <limit
-          effort="91.0"
-          velocity="100.7"/>
+          effort="108.6"
+          velocity="36.65"/>
     </joint>
     <link name="right_motor">
@@ -223,5 +224,8 @@
         <child link="front_right_wheel_hub"/>
         <axis xyz="0 0 -1"/>
-        <limit effort="100" velocity="20" lower="-0.4" upper="0.4"/>
+        <limit  effort="33.4"
+          velocity="1.745"
+          lower="-1.308"
+          upper="1.308"/>
           <dynamics damping="0.1" friction="0.05"/>
     </joint>
@@ -287,5 +291,8 @@
         <child link="front_left_wheel_hub"/>
         <axis xyz="0 0 -1"/>
-         <limit effort="100" velocity="20" lower="-0.4" upper="0.4"/>
+         <limit  effort="33.4"
+          velocity="1.745"
+          lower="-1.308"
+          upper="1.308"/>
           <dynamics damping="0.1" friction="0.05"/>
     </joint>

File: src/avone/description/ros2_control_hardware.xacro (robot description, xacro)
@@ -4,16 +4,17 @@
     <hardware>
       <plugin>avone/AvoneSystemHardware</plugin>
-      <param name="max_steer_angle">0.7</param>
-      <param name="min_steer_angle">-0.7</param>
-      <param name="max_rpm">15000</param>
-      <param name="can_interface">vcan0</param>
+      <param name="max_steer_angle">1.3</param>
+      <param name="min_steer_angle">-1.3</param>
+      <param name="max_rpm">350</param>
+      <param name="can_interface">can0</param>
       <param name="can_baudrate">250000</param>
       <param name="read_timeout_ms">20</param>
-      <param name="l_motor_can_id">0x127</param>
-      <param name="r_motor_can_id">0x128</param>
-      <param name="steer_can_id">0x200</param>
-      <param name="cmd_l_motor_can_id">0x27</param>
-      <param name="cmd_r_motor_can_id">0x28</param>
-      <param name="cmd_steer_can_id">0x20</param>
+      <param name="l_motor_can_id">0x8CF11E05</param>
+      <!-- set right as same as left until figure out motor controller  -->
+      <param name="r_motor_can_id">0x8CF11E06</param>
+      <param name="steer_can_id">0x006</param>
+      <param name="cmd_l_motor_can_id">0x0B</param>
+      <param name="cmd_r_motor_can_id">0x0C</param>
+      <param name="cmd_steer_can_id">0x004</param>
     </hardware>
   <!-- front steering -->

Commit message: updated meshes to package instead of local

File: src/avone/description/robot_core.xacro (robot description, xacro)
@@ -36,6 +36,6 @@
             <origin xyz="2.2924 -0.00985747 0.0751" rpy="3.14159 0 1.5708"/>
             <geometry>
-                  <mesh filename="file:///home/jay/ros2_ws/src/avone/description/assets/chassis.stl"/>
-                 <!-- <mesh filename="package://avone/description/assets/chassis.stl"/> -->
+                  <mesh filename="package://avone/description/assets/chassis.stl"/>
+                  <!-- <mesh filename="file:///home/jay/ros2_ws/src/avone/description/assets/chassis.stl"/> -->
                  <!--  <box size="0.3 0.3 0.15"/> -->
             </geometry>
@@ -45,5 +45,5 @@
             <origin xyz="2.2924 -0.00985747 0.0751" rpy="3.14159 0 1.5708"/>
             <geometry>
-                    <mesh filename="file:///home/jay/ros2_ws/src/avone/description/assets/chassis.stl"/>
+                    <mesh filename="package://avone/description/assets/chassis.stl"/>
                  <!--  <box size="0.3 0.3 0.15"/> -->
             </geometry>
@@ -56,5 +56,5 @@
       <origin xyz="-0.170629 -0.28192 0.105" rpy="3.14159 5.47382e-48 -0.0851102"/>
       <geometry>
-        <mesh filename="file:///home/jay/ros2_ws/src/avone/description/assets/rear_suspension.stl"/>
+        <mesh filename="package://avone/description/assets/rear_suspension.stl"/>
       </geometry>
       <material name="blue"/>
@@ -63,5 +63,5 @@
       <origin xyz="-0.170629 -0.28192 0.105" rpy="3.14159 5.47382e-48 -0.0851102"/>
       <geometry>
-        <mesh filename="file:///home/jay/ros2_ws/src/avone/description/assets/rear_suspension.stl"/>
+        <mesh filename="package://avone/description/assets/rear_suspension.stl"/>
       </geometry>
     </collision>
@@ -70,5 +70,5 @@
       <origin xyz="0.189017 0.312761 0.105" rpy="-3.14159 2.33363e-61 -3.05648"/>
       <geometry>
-        <mesh filename="file:///home/jay/ros2_ws/src/avone/description/assets/rear_suspension.stl"/>
+        <mesh filename="package://avone/description/assets/rear_suspension.stl"/>
       </geometry>
       <material name="blue"/>
@@ -77,5 +77,5 @@
       <origin xyz="0.189017 0.312761 0.105" rpy="-3.14159 2.33363e-61 -3.05648"/>
       <geometry>
-        <mesh filename="file:///home/jay/ros2_ws/src/avone/description/assets/rear_suspension.stl"/>
+        <mesh filename="package://avone/description/assets/rear_suspension.stl"/>
       </geometry>
     </collision>
@@ -84,5 +84,5 @@
       <origin xyz="1.6032 0.2935 0.075" rpy="3.14159 -1.54112e-16 1.5708"/>
       <geometry>
-        <mesh filename="file:///home/jay/ros2_ws/src/avone/description/assets/front_suspension.stl"/>
+        <mesh filename="package://avone/description/assets/front_suspension.stl"/>
       </geometry>
       <material name="blue"/>
@@ -91,5 +91,5 @@
       <origin xyz="1.6032 0.2935 0.075" rpy="3.14159 -1.54112e-16 1.5708"/>
       <geometry>
-        <mesh filename="file:///home/jay/ros2_ws/src/avone/description/assets/front_suspension.stl"/>
+        <mesh filename="package://avone/description/assets/front_suspension.stl"/>
       </geometry>
     </collision>
@@ -98,5 +98,5 @@
       <origin xyz="1.8748 -0.2935 0.075" rpy="-3.14159 1.54112e-16 -1.5708"/>
       <geometry>
-        <mesh filename="file:///home/jay/ros2_ws/src/avone/description/assets/front_suspension.stl"/>
+        <mesh filename="package://avone/description/assets/front_suspension.stl"/>
       </geometry>
       <material name="blue"/>
@@ -105,5 +105,5 @@
       <origin xyz="1.8748 -0.2935 0.075" rpy="-3.14159 1.54112e-16 -1.5708"/>
       <geometry>
-        <mesh filename="file:///home/jay/ros2_ws/src/avone/description/assets/front_suspension.stl"/>
+        <mesh filename="package://avone/description/assets/front_suspension.stl"/>
       </geometry>
     </collision>
@@ -112,5 +112,5 @@
       <origin xyz="-0.181377 0.297001 -0.105" rpy="6.30462e-15 0 -6.18615e-05"/>
       <geometry>
-        <mesh filename="file:///home/jay/ros2_ws/src/avone/description/assets/rear_wheel_hub.stl"/>
+        <mesh filename="package://avone/description/assets/rear_wheel_hub.stl"/>
       </geometry>
       <material name="white"/>
@@ -119,5 +119,5 @@
       <origin xyz="-0.181377 0.297001 -0.105" rpy="6.30462e-15 0 -6.18615e-05"/>
       <geometry>
-        <mesh filename="file:///home/jay/ros2_ws/src/avone/description/assets/rear_wheel_hub.stl"/>
+        <mesh filename="package://avone/description/assets/rear_wheel_hub.stl"/>
       </geometry>
     </collision>
@@ -126,5 +126,5 @@
       <origin xyz="0.181423 -0.296978 -0.105" rpy="3.10966e-15 7.00787e-15 -3.14153"/>
       <geometry>
-        <mesh filename="file:///home/jay/ros2_ws/src/avone/description/assets/rear_wheel_hub.stl"/>
+        <mesh filename="package://avone/description/assets/rear_wheel_hub.stl"/>
       </geometry>
       <material name="white"/>
@@ -133,5 +133,5 @@
       <origin xyz="0.181423 -0.296978 -0.105" rpy="3.10966e-15 7.00787e-15 -3.14153"/>
       <geometry>
-        <mesh filename="file:///home/jay/ros2_ws/src/avone/description/assets/rear_wheel_hub.stl"/>
+        <mesh filename="package://avone/description/assets/rear_wheel_hub.stl"/>
       </geometry>
     </collision>
@@ -163,5 +163,5 @@
             <origin xyz="-8.09391e-17 7.65875e-18 0.17" rpy="1.5708 0 0"/>
             <geometry>
-                    <mesh filename="file:///home/jay/ros2_ws/src/avone/description/assets/wheel.stl"/>
+                    <mesh filename="package://avone/description/assets/wheel.stl"/>
                  <!--  <box size="0.3 0.3 0.15"/> -->
             </geometry>
@@ -171,5 +171,5 @@
             <origin xyz="-8.09391e-17 7.65875e-18 0.17" rpy="1.5708 0 0"/>
             <geometry>
-                     <!--<mesh filename="file:///home/jay/ros2_ws/src/avone/description/assets/wheel.stl"/>    -->
+                     <!--<mesh filename="package://avone/description/assets/wheel.stl"/>    -->
                                         <sphere radius="0.203"/>
                  <!--  <box size="0.3 0.3 0.15"/> -->
@@ -198,5 +198,5 @@
             <origin xyz="-1.59877e-17 7.65404e-18 0.17" rpy="1.5708 0 0"/>
             <geometry>
-                    <mesh filename="file:///home/jay/ros2_ws/src/avone/description/assets/wheel.stl"/>
+                    <mesh filename="package://avone/description/assets/wheel.stl"/>
                  <!--  <box size="0.3 0.3 0.15"/> -->
             </geometry>
@@ -234,5 +234,5 @@
             <origin xyz="-0.290639 0.1358 0.18" rpy="-3.14159 0 0"/>
             <geometry>
-                    <mesh filename="file:///home/jay/ros2_ws/src/avone/description/assets/front_wheel_hub.stl"/>
+                    <mesh filename="package://avone/description/assets/front_wheel_hub.stl"/>
                  <!--  <box size="0.3 0.3 0.15"/> -->
             </geometry>
@@ -242,5 +242,5 @@
             <origin xyz="-0.290639 0.1358 0.18" rpy="-3.14159 0 0"/>
             <geometry>
-                    <mesh filename="file:///home/jay/ros2_ws/src/avone/description/assets/front_wheel_hub.stl"/>
+                    <mesh filename="package://avone/description/assets/front_wheel_hub.stl"/>
                  <!--  <box size="0.3 0.3 0.15"/> -->
             </geometry>
@@ -265,5 +265,5 @@
             <origin xyz="2.22045e-16 0 0.17" rpy="1.5708 0 1.5708"/>
             <geometry>
-                    <mesh filename="file:///home/jay/ros2_ws/src/avone/description/assets/wheel.stl"/>
+                    <mesh filename="package://avone/description/assets/wheel.stl"/>
                  <!--  <box size="0.3 0.3 0.15"/> -->
             </geometry>
@@ -273,5 +273,5 @@
             <origin xyz="2.22045e-16 0 0.17" rpy="1.5708 0 1.5708"/>
             <geometry>
-                   <!--<mesh filename="file:///home/jay/ros2_ws/src/avone/description/assets/wheel.stl"/>    -->
+                   <!--<mesh filename="package://avone/description/assets/wheel.stl"/>    -->
                                         <sphere radius="0.203"/>
                  <!--  <box size="0.3 0.3 0.15"/> -->
@@ -301,5 +301,5 @@
         <origin xyz="-0.290639 0.1358 0.18" rpy="3.14159 0 0"/>
         <geometry>
-                    <mesh filename="file:///home/jay/ros2_ws/src/avone/description/assets/front_wheel_hub.stl"/>
+                    <mesh filename="package://avone/description/assets/front_wheel_hub.stl"/>
                  <!--  <box size="0.3 0.3 0.15"/> -->
         </geometry>
@@ -309,5 +309,5 @@
         <origin xyz="-0.290639 0.1358 0.18" rpy="3.14159 0 0"/>
         <geometry>
-                    <mesh filename="file:///home/jay/ros2_ws/src/avone/description/assets/front_wheel_hub.stl"/>
+                    <mesh filename="package://avone/description/assets/front_wheel_hub.stl"/>
                  <!--  <box size="0.3 0.3 0.15"/> -->
         </geometry>
@@ -332,5 +332,5 @@
         <origin xyz="0 0 0.17" rpy="1.5708 0 0"/>
         <geometry>
-                    <mesh filename="file:///home/jay/ros2_ws/src/avone/description/assets/wheel.stl"/>
+                    <mesh filename="package://avone/description/assets/wheel.stl"/>
                  <!--  <box size="0.3 0.3 0.15"/> -->
         </geometry>
@@ -340,5 +340,5 @@
         <origin xyz="0 0 0.17" rpy="1.5708 0 0"/>
         <geometry>
-                      <!--<mesh filename="file:///home/jay/ros2_ws/src/avone/description/assets/wheel.stl"/>    -->
+                      <!--<mesh filename="package://avone/description/assets/wheel.stl"/>    -->
                                         <sphere radius="0.203"/>
                  <!--  <box size="0.3 0.3 0.15"/> -->
