Commit message: final push from NUC after final test day - before clean and finalise

File: src/avone/description/robot_core.xacro (robot description, xacro)
@@ -3,5 +3,5 @@
     <xacro:include filename="inertial_macros.xacro"/>
     <!-- change this to local directroy -->
-    <!-- <xacro:arg name="mesh_dir" default="file://home/jay/ros2_ws/src/avone/description/assets"/> -->
+    <!-- <xacro:arg name="mesh_dir" default="file://home/avone/avone_ws/src/avone/description/assets"/> -->
     <material name="white">
         <color rgba="1 1 1 1" />
@@ -38,7 +38,7 @@
             <origin xyz="2.2924 -0.00985747 0.0751" rpy="3.14159 0 1.5708"/>
             <geometry>
-                  <!-- <mesh filename="file:///home/jay/ros2_ws/src/avone/description/assets/chassis.stl"/> -->
-                  <mesh filename="file:///home/jay/ros2_ws/src/avone/description/assets/chassis.stl"/>
-<!-- home/jay/ros2_ws/src/avone -->
+                  <!-- <mesh filename="file:///home/avone/avone_ws/src/avone/description/assets/chassis.stl"/> -->
+                  <mesh filename="file:///home/avone/avone_ws/src/avone/description/assets/chassis.stl"/>
+<!-- home/avone/avone_ws/src/avone -->
                  <!--  <box size="0.3 0.3 0.15"/> -->
             </geometry>
@@ -48,5 +48,5 @@
             <origin xyz="2.2924 -0.00985747 0.0751" rpy="3.14159 0 1.5708"/>
             <geometry>
-                    <mesh filename="file:///home/jay/ros2_ws/src/avone/description/assets/chassis.stl"/>
+                    <mesh filename="file:///home/avone/avone_ws/src/avone/description/assets/chassis.stl"/>
                  <!--  <box size="0.3 0.3 0.15"/> -->
             </geometry>
@@ -59,5 +59,5 @@
       <origin xyz="-0.170629 -0.28192 0.105" rpy="3.14159 5.47382e-48 -0.0851102"/>
       <geometry>
-        <mesh filename="file:///home/jay/ros2_ws/src/avone/description/assets/rear_suspension.stl"/>
+        <mesh filename="file:///home/avone/avone_ws/src/avone/description/assets/rear_suspension.stl"/>
       </geometry>
       <material name="blue"/>
@@ -66,5 +66,5 @@
       <origin xyz="-0.170629 -0.28192 0.105" rpy="3.14159 5.47382e-48 -0.0851102"/>
       <geometry>
-        <mesh filename="file:///home/jay/ros2_ws/src/avone/description/assets/rear_suspension.stl"/>
+        <mesh filename="file:///home/avone/avone_ws/src/avone/description/assets/rear_suspension.stl"/>
       </geometry>
     </collision>
@@ -73,5 +73,5 @@
       <origin xyz="0.189017 0.312761 0.105" rpy="-3.14159 2.33363e-61 -3.05648"/>
       <geometry>
-        <mesh filename="file:///home/jay/ros2_ws/src/avone/description/assets/rear_suspension.stl"/>
+        <mesh filename="file:///home/avone/avone_ws/src/avone/description/assets/rear_suspension.stl"/>
       </geometry>
       <material name="blue"/>
@@ -80,5 +80,5 @@
       <origin xyz="0.189017 0.312761 0.105" rpy="-3.14159 2.33363e-61 -3.05648"/>
       <geometry>
-        <mesh filename="file:///home/jay/ros2_ws/src/avone/description/assets/rear_suspension.stl"/>
+        <mesh filename="file:///home/avone/avone_ws/src/avone/description/assets/rear_suspension.stl"/>
       </geometry>
     </collision>
@@ -87,5 +87,5 @@
       <origin xyz="1.6032 0.2935 0.075" rpy="3.14159 -1.54112e-16 1.5708"/>
       <geometry>
-        <mesh filename="file:///home/jay/ros2_ws/src/avone/description/assets/front_suspension.stl"/>
+        <mesh filename="file:///home/avone/avone_ws/src/avone/description/assets/front_suspension.stl"/>
       </geometry>
       <material name="blue"/>
@@ -94,5 +94,5 @@
       <origin xyz="1.6032 0.2935 0.075" rpy="3.14159 -1.54112e-16 1.5708"/>
       <geometry>
-        <mesh filename="file:///home/jay/ros2_ws/src/avone/description/assets/front_suspension.stl"/>
+        <mesh filename="file:///home/avone/avone_ws/src/avone/description/assets/front_suspension.stl"/>
       </geometry>
     </collision>
@@ -101,5 +101,5 @@
       <origin xyz="1.8748 -0.2935 0.075" rpy="-3.14159 1.54112e-16 -1.5708"/>
       <geometry>
-        <mesh filename="file:///home/jay/ros2_ws/src/avone/description/assets/front_suspension.stl"/>
+        <mesh filename="file:///home/avone/avone_ws/src/avone/description/assets/front_suspension.stl"/>
       </geometry>
       <material name="blue"/>
@@ -108,5 +108,5 @@
       <origin xyz="1.8748 -0.2935 0.075" rpy="-3.14159 1.54112e-16 -1.5708"/>
       <geometry>
-        <mesh filename="file:///home/jay/ros2_ws/src/avone/description/assets/front_suspension.stl"/>
+        <mesh filename="file:///home/avone/avone_ws/src/avone/description/assets/front_suspension.stl"/>
       </geometry>
     </collision>
@@ -115,5 +115,5 @@
       <origin xyz="-0.181377 0.297001 -0.105" rpy="6.30462e-15 0 -6.18615e-05"/>
       <geometry>
-        <mesh filename="file:///home/jay/ros2_ws/src/avone/description/assets/rear_wheel_hub.stl"/>
+        <mesh filename="file:///home/avone/avone_ws/src/avone/description/assets/rear_wheel_hub.stl"/>
       </geometry>
       <material name="white"/>
@@ -122,5 +122,5 @@
       <origin xyz="-0.181377 0.297001 -0.105" rpy="6.30462e-15 0 -6.18615e-05"/>
       <geometry>
-        <mesh filename="file:///home/jay/ros2_ws/src/avone/description/assets/rear_wheel_hub.stl"/>
+        <mesh filename="file:///home/avone/avone_ws/src/avone/description/assets/rear_wheel_hub.stl"/>
       </geometry>
     </collision>
@@ -129,5 +129,5 @@
       <origin xyz="0.181423 -0.296978 -0.105" rpy="3.10966e-15 7.00787e-15 -3.14153"/>
       <geometry>
-        <mesh filename="file:///home/jay/ros2_ws/src/avone/description/assets/rear_wheel_hub.stl"/>
+        <mesh filename="file:///home/avone/avone_ws/src/avone/description/assets/rear_wheel_hub.stl"/>
       </geometry>
       <material name="white"/>
@@ -136,5 +136,5 @@
       <origin xyz="0.181423 -0.296978 -0.105" rpy="3.10966e-15 7.00787e-15 -3.14153"/>
       <geometry>
-        <mesh filename="file:///home/jay/ros2_ws/src/avone/description/assets/rear_wheel_hub.stl"/>
+        <mesh filename="file:///home/avone/avone_ws/src/avone/description/assets/rear_wheel_hub.stl"/>
       </geometry>
     </collision>
@@ -166,5 +166,5 @@
             <origin xyz="-8.09391e-17 7.65875e-18 0.17" rpy="1.5708 0 0"/>
             <geometry>
-                    <mesh filename="file:///home/jay/ros2_ws/src/avone/description/assets/wheel.stl"/>
+                    <mesh filename="file:///home/avone/avone_ws/src/avone/description/assets/wheel.stl"/>
                  <!--  <box size="0.3 0.3 0.15"/> -->
             </geometry>
@@ -174,5 +174,5 @@
             <origin xyz="-8.09391e-17 7.65875e-18 0.17" rpy="1.5708 0 0"/>
             <geometry>
-                     <!--<mesh filename="file:///home/jay/ros2_ws/src/avone/description/assets/wheel.stl"/>    -->
+                     <!--<mesh filename="file:///home/avone/avone_ws/src/avone/description/assets/wheel.stl"/>    -->
                                         <sphere radius="0.203"/>
                  <!--  <box size="0.3 0.3 0.15"/> -->
@@ -201,5 +201,5 @@
             <origin xyz="-1.59877e-17 7.65404e-18 0.17" rpy="1.5708 0 0"/>
             <geometry>
-                    <mesh filename="file:///home/jay/ros2_ws/src/avone/description/assets/wheel.stl"/>
+                    <mesh filename="file:///home/avone/avone_ws/src/avone/description/assets/wheel.stl"/>
                  <!--  <box size="0.3 0.3 0.15"/> -->
             </geometry>
@@ -237,5 +237,5 @@
             <origin xyz="-0.290639 0.1358 0.18" rpy="-3.14159 0 0"/>
             <geometry>
-                    <mesh filename="file:///home/jay/ros2_ws/src/avone/description/assets/front_wheel_hub.stl"/>
+                    <mesh filename="file:///home/avone/avone_ws/src/avone/description/assets/front_wheel_hub.stl"/>
                  <!--  <box size="0.3 0.3 0.15"/> -->
             </geometry>
@@ -245,5 +245,5 @@
             <origin xyz="-0.290639 0.1358 0.18" rpy="-3.14159 0 0"/>
             <geometry>
-                    <mesh filename="file:///home/jay/ros2_ws/src/avone/description/assets/front_wheel_hub.stl"/>
+                    <mesh filename="file:///home/avone/avone_ws/src/avone/description/assets/front_wheel_hub.stl"/>
                  <!--  <box size="0.3 0.3 0.15"/> -->
             </geometry>
@@ -268,5 +268,5 @@
             <origin xyz="2.22045e-16 0 0.17" rpy="1.5708 0 1.5708"/>
             <geometry>
-                    <mesh filename="file:///home/jay/ros2_ws/src/avone/description/assets/wheel.stl"/>
+                    <mesh filename="file:///home/avone/avone_ws/src/avone/description/assets/wheel.stl"/>
                  <!--  <box size="0.3 0.3 0.15"/> -->
             </geometry>
@@ -276,5 +276,5 @@
             <origin xyz="2.22045e-16 0 0.17" rpy="1.5708 0 1.5708"/>
             <geometry>
-                   <!--<mesh filename="file:///home/jay/ros2_ws/src/avone/description/assets/wheel.stl"/>    -->
+                   <!--<mesh filename="file:///home/avone/avone_ws/src/avone/description/assets/wheel.stl"/>    -->
                                         <sphere radius="0.203"/>
                  <!--  <box size="0.3 0.3 0.15"/> -->
@@ -304,5 +304,5 @@
         <origin xyz="-0.290639 0.1358 0.18" rpy="3.14159 0 0"/>
         <geometry>
-                    <mesh filename="file:///home/jay/ros2_ws/src/avone/description/assets/front_wheel_hub.stl"/>
+                    <mesh filename="file:///home/avone/avone_ws/src/avone/description/assets/front_wheel_hub.stl"/>
                  <!--  <box size="0.3 0.3 0.15"/> -->
         </geometry>
@@ -312,5 +312,5 @@
         <origin xyz="-0.290639 0.1358 0.18" rpy="3.14159 0 0"/>
         <geometry>
-                    <mesh filename="file:///home/jay/ros2_ws/src/avone/description/assets/front_wheel_hub.stl"/>
+                    <mesh filename="file:///home/avone/avone_ws/src/avone/description/assets/front_wheel_hub.stl"/>
                  <!--  <box size="0.3 0.3 0.15"/> -->
         </geometry>
@@ -335,5 +335,5 @@
         <origin xyz="0 0 0.17" rpy="1.5708 0 0"/>
         <geometry>
-                    <mesh filename="file:///home/jay/ros2_ws/src/avone/description/assets/wheel.stl"/>
+                    <mesh filename="file:///home/avone/avone_ws/src/avone/description/assets/wheel.stl"/>
                  <!--  <box size="0.3 0.3 0.15"/> -->
         </geometry>
@@ -343,5 +343,5 @@
         <origin xyz="0 0 0.17" rpy="1.5708 0 0"/>
         <geometry>
-                      <!--<mesh filename="file:///home/jay/ros2_ws/src/avone/description/assets/wheel.stl"/>    -->
+                      <!--<mesh filename="file:///home/avone/avone_ws/src/avone/description/assets/wheel.stl"/>    -->
                                         <sphere radius="0.203"/>
                  <!--  <box size="0.3 0.3 0.15"/> -->

File: src/avone/description/sensors.xacro (robot description, xacro)
@@ -20,5 +20,5 @@
         <parent link="chassis"/>
         <child link="gps_link1"/>
-          <origin xyz="-0.1188 0 0.3924" rpy="0 0 0"/>
+          <origin xyz="-0.107 0 0.4434" rpy="0 0 0"/>
     </joint>
   <link name="gps_link1">
@@ -50,5 +50,5 @@
         <parent link="chassis"/>
         <child link="gps_link2"/>
-          <origin xyz="2.131 0 0.3924" rpy="0 0 0"/>
+          <origin xyz="1.693 0 0.4434" rpy="0 0 0"/>
     </joint>
   <link name="gps_link2">

Commit message: commit before final clean

File: src/avone/description/robot_core.xacro (robot description, xacro)
@@ -2,6 +2,7 @@
 <robot xmlns:xacro="http://www.ros.org/wiki/xacro" >
     <xacro:include filename="inertial_macros.xacro"/>
-    <!-- change this to local directroy -->
-    <!-- <xacro:arg name="mesh_dir" default="file://home/avone/avone_ws/src/avone/description/assets"/> -->
+    <!-- FOR GAZEBO SIM - CHANGE MESH TO FULL PATH - EG: -->
+    <!-- Replace package:// with file:///home/avone/avone_ws/src/ (user and folder dependant)-->
+    <!-- <mesh filename="file:///home/avone/avone_ws/src/avone/description/assets/chassis.stl"/> -->
     <material name="white">
         <color rgba="1 1 1 1" />
@@ -38,8 +39,5 @@
             <origin xyz="2.2924 -0.00985747 0.0751" rpy="3.14159 0 1.5708"/>
             <geometry>
-                  <!-- <mesh filename="file:///home/avone/avone_ws/src/avone/description/assets/chassis.stl"/> -->
-                  <mesh filename="file:///home/avone/avone_ws/src/avone/description/assets/chassis.stl"/>
-<!-- home/avone/avone_ws/src/avone -->
-                 <!--  <box size="0.3 0.3 0.15"/> -->
+                  <mesh filename="package://avone/description/assets/chassis.stl"/>
             </geometry>
             <material name="blue"/>
@@ -48,6 +46,5 @@
             <origin xyz="2.2924 -0.00985747 0.0751" rpy="3.14159 0 1.5708"/>
             <geometry>
-                    <mesh filename="file:///home/avone/avone_ws/src/avone/description/assets/chassis.stl"/>
-                 <!--  <box size="0.3 0.3 0.15"/> -->
+                    <mesh filename="package://avone/description/assets/chassis.stl"/>
             </geometry>
         </collision>
@@ -59,5 +56,5 @@
       <origin xyz="-0.170629 -0.28192 0.105" rpy="3.14159 5.47382e-48 -0.0851102"/>
       <geometry>
-        <mesh filename="file:///home/avone/avone_ws/src/avone/description/assets/rear_suspension.stl"/>
+        <mesh filename="package://avone/description/assets/rear_suspension.stl"/>
       </geometry>
       <material name="blue"/>
@@ -66,5 +63,5 @@
       <origin xyz="-0.170629 -0.28192 0.105" rpy="3.14159 5.47382e-48 -0.0851102"/>
       <geometry>
-        <mesh filename="file:///home/avone/avone_ws/src/avone/description/assets/rear_suspension.stl"/>
+        <mesh filename="package://avone/description/assets/rear_suspension.stl"/>
       </geometry>
     </collision>
@@ -73,5 +70,5 @@
       <origin xyz="0.189017 0.312761 0.105" rpy="-3.14159 2.33363e-61 -3.05648"/>
       <geometry>
-        <mesh filename="file:///home/avone/avone_ws/src/avone/description/assets/rear_suspension.stl"/>
+        <mesh filename="package://avone/description/assets/rear_suspension.stl"/>
       </geometry>
       <material name="blue"/>
@@ -80,5 +77,5 @@
       <origin xyz="0.189017 0.312761 0.105" rpy="-3.14159 2.33363e-61 -3.05648"/>
       <geometry>
-        <mesh filename="file:///home/avone/avone_ws/src/avone/description/assets/rear_suspension.stl"/>
+        <mesh filename="package://avone/description/assets/rear_suspension.stl"/>
       </geometry>
     </collision>
@@ -87,5 +84,5 @@
       <origin xyz="1.6032 0.2935 0.075" rpy="3.14159 -1.54112e-16 1.5708"/>
       <geometry>
-        <mesh filename="file:///home/avone/avone_ws/src/avone/description/assets/front_suspension.stl"/>
+        <mesh filename="package://avone/description/assets/front_suspension.stl"/>
       </geometry>
       <material name="blue"/>
@@ -94,5 +91,5 @@
       <origin xyz="1.6032 0.2935 0.075" rpy="3.14159 -1.54112e-16 1.5708"/>
       <geometry>
-        <mesh filename="file:///home/avone/avone_ws/src/avone/description/assets/front_suspension.stl"/>
+        <mesh filename="package://avone/description/assets/front_suspension.stl"/>
       </geometry>
     </collision>
@@ -101,5 +98,5 @@
       <origin xyz="1.8748 -0.2935 0.075" rpy="-3.14159 1.54112e-16 -1.5708"/>
       <geometry>
-        <mesh filename="file:///home/avone/avone_ws/src/avone/description/assets/front_suspension.stl"/>
+        <mesh filename="package://avone/description/assets/front_suspension.stl"/>
       </geometry>
       <material name="blue"/>
@@ -108,5 +105,5 @@
       <origin xyz="1.8748 -0.2935 0.075" rpy="-3.14159 1.54112e-16 -1.5708"/>
       <geometry>
-        <mesh filename="file:///home/avone/avone_ws/src/avone/description/assets/front_suspension.stl"/>
+        <mesh filename="package://avone/description/assets/front_suspension.stl"/>
       </geometry>
     </collision>
@@ -115,5 +112,5 @@
       <origin xyz="-0.181377 0.297001 -0.105" rpy="6.30462e-15 0 -6.18615e-05"/>
       <geometry>
-        <mesh filename="file:///home/avone/avone_ws/src/avone/description/assets/rear_wheel_hub.stl"/>
+        <mesh filename="package://avone/description/assets/rear_wheel_hub.stl"/>
       </geometry>
       <material name="white"/>
@@ -122,5 +119,5 @@
       <origin xyz="-0.181377 0.297001 -0.105" rpy="6.30462e-15 0 -6.18615e-05"/>
       <geometry>
-        <mesh filename="file:///home/avone/avone_ws/src/avone/description/assets/rear_wheel_hub.stl"/>
+        <mesh filename="package://avone/description/assets/rear_wheel_hub.stl"/>
       </geometry>
     </collision>
@@ -129,5 +126,5 @@
       <origin xyz="0.181423 -0.296978 -0.105" rpy="3.10966e-15 7.00787e-15 -3.14153"/>
       <geometry>
-        <mesh filename="file:///home/avone/avone_ws/src/avone/description/assets/rear_wheel_hub.stl"/>
+        <mesh filename="package://avone/description/assets/rear_wheel_hub.stl"/>
       </geometry>
       <material name="white"/>
@@ -136,5 +133,5 @@
       <origin xyz="0.181423 -0.296978 -0.105" rpy="3.10966e-15 7.00787e-15 -3.14153"/>
       <geometry>
-        <mesh filename="file:///home/avone/avone_ws/src/avone/description/assets/rear_wheel_hub.stl"/>
+        <mesh filename="package://avone/description/assets/rear_wheel_hub.stl"/>
       </geometry>
     </collision>
@@ -166,5 +163,5 @@
             <origin xyz="-8.09391e-17 7.65875e-18 0.17" rpy="1.5708 0 0"/>
             <geometry>
-                    <mesh filename="file:///home/avone/avone_ws/src/avone/description/assets/wheel.stl"/>
+                    <mesh filename="package://avone/description/assets/wheel.stl"/>
                  <!--  <box size="0.3 0.3 0.15"/> -->
             </geometry>
@@ -174,5 +171,5 @@
             <origin xyz="-8.09391e-17 7.65875e-18 0.17" rpy="1.5708 0 0"/>
             <geometry>
-                     <!--<mesh filename="file:///home/avone/avone_ws/src/avone/description/assets/wheel.stl"/>    -->
+                     <!--<mesh filename="package://avone/description/assets/wheel.stl"/>    -->
                                         <sphere radius="0.203"/>
                  <!--  <box size="0.3 0.3 0.15"/> -->
@@ -201,5 +198,5 @@
             <origin xyz="-1.59877e-17 7.65404e-18 0.17" rpy="1.5708 0 0"/>
             <geometry>
-                    <mesh filename="file:///home/avone/avone_ws/src/avone/description/assets/wheel.stl"/>
+                    <mesh filename="package://avone/description/assets/wheel.stl"/>
                  <!--  <box size="0.3 0.3 0.15"/> -->
             </geometry>
@@ -237,5 +234,5 @@
             <origin xyz="-0.290639 0.1358 0.18" rpy="-3.14159 0 0"/>
             <geometry>
-                    <mesh filename="file:///home/avone/avone_ws/src/avone/description/assets/front_wheel_hub.stl"/>
+                    <mesh filename="package://avone/description/assets/front_wheel_hub.stl"/>
                  <!--  <box size="0.3 0.3 0.15"/> -->
             </geometry>
@@ -245,5 +242,5 @@
             <origin xyz="-0.290639 0.1358 0.18" rpy="-3.14159 0 0"/>
             <geometry>
-                    <mesh filename="file:///home/avone/avone_ws/src/avone/description/assets/front_wheel_hub.stl"/>
+                    <mesh filename="package://avone/description/assets/front_wheel_hub.stl"/>
                  <!--  <box size="0.3 0.3 0.15"/> -->
             </geometry>
@@ -268,5 +265,5 @@
             <origin xyz="2.22045e-16 0 0.17" rpy="1.5708 0 1.5708"/>
             <geometry>
-                    <mesh filename="file:///home/avone/avone_ws/src/avone/description/assets/wheel.stl"/>
+                    <mesh filename="package://avone/description/assets/wheel.stl"/>
                  <!--  <box size="0.3 0.3 0.15"/> -->
             </geometry>
@@ -276,5 +273,5 @@
             <origin xyz="2.22045e-16 0 0.17" rpy="1.5708 0 1.5708"/>
             <geometry>
-                   <!--<mesh filename="file:///home/avone/avone_ws/src/avone/description/assets/wheel.stl"/>    -->
+                   <!--<mesh filename="package://avone/description/assets/wheel.stl"/>    -->
                                         <sphere radius="0.203"/>
                  <!--  <box size="0.3 0.3 0.15"/> -->
@@ -304,5 +301,5 @@
         <origin xyz="-0.290639 0.1358 0.18" rpy="3.14159 0 0"/>
         <geometry>
-                    <mesh filename="file:///home/avone/avone_ws/src/avone/description/assets/front_wheel_hub.stl"/>
+                    <mesh filename="package://avone/description/assets/front_wheel_hub.stl"/>
                  <!--  <box size="0.3 0.3 0.15"/> -->
         </geometry>
@@ -312,5 +309,5 @@
         <origin xyz="-0.290639 0.1358 0.18" rpy="3.14159 0 0"/>
         <geometry>
-                    <mesh filename="file:///home/avone/avone_ws/src/avone/description/assets/front_wheel_hub.stl"/>
+                    <mesh filename="package://avone/description/assets/front_wheel_hub.stl"/>
                  <!--  <box size="0.3 0.3 0.15"/> -->
         </geometry>
@@ -335,5 +332,5 @@
         <origin xyz="0 0 0.17" rpy="1.5708 0 0"/>
         <geometry>
-                    <mesh filename="file:///home/avone/avone_ws/src/avone/description/assets/wheel.stl"/>
+                    <mesh filename="package://avone/description/assets/wheel.stl"/>
                  <!--  <box size="0.3 0.3 0.15"/> -->
         </geometry>
@@ -343,5 +340,5 @@
         <origin xyz="0 0 0.17" rpy="1.5708 0 0"/>
         <geometry>
-                      <!--<mesh filename="file:///home/avone/avone_ws/src/avone/description/assets/wheel.stl"/>    -->
+                      <!--<mesh filename="package://avone/description/assets/wheel.stl"/>    -->
                                         <sphere radius="0.203"/>
                  <!--  <box size="0.3 0.3 0.15"/> -->
