Commit message: addition of cone landmark code and pointcloud filtering

File: src/avone/description/camera.xacro (robot description, xacro)
@@ -23,20 +23,20 @@
         <material>Gazebo/Red</material>
         <sensor name="camera" type="camera">
-            <gz_frame_id>camera_link_optical</gz_frame_id>
+            <gz_frame_id>camera_link</gz_frame_id>
             <pose> 0 0 0 0 0 0 </pose>
             <visualize>true</visualize>
-            <update_rate>10</update_rate>
+            <update_rate>30</update_rate>
             <topic>camera/image_raw</topic>
             <camera>
             <camera_info_topic>camera/camera_info</camera_info_topic>
-                <horizontal_fov>1.089</horizontal_fov>
+                      <horizontal_fov>1.91986</horizontal_fov>
                 <image>
                     <format>R8G8B8</format>
-                    <width>1920</width>
-                    <height>1080</height>
+                    <width>1280</width>
+                    <height>720</height>
                 </image>
                 <clip>
-                    <near>0.05</near>
-                    <far>50.0</far>
+                    <near>0.3</near>
+                    <far>20.0</far>
                 </clip>
             </camera>

File: src/avone/description/lidar.xacro (robot description, xacro)
@@ -4,5 +4,5 @@
         <parent link="chassis"/>
         <child link="laser_frame"/>
-        <origin xyz="2.4174 0 -0.11" rpy="0 0 0"/>
+        <origin xyz="2.4174 0 0.2977" rpy="0 0 0"/>
     </joint>
     <link name="laser_frame">
@@ -45,13 +45,13 @@
                     </horizontal>
                     <vertical>
-                        <samples>1</samples>
-                        <resolution>0.01</resolution>
-                        <min_angle>0</min_angle>
-                        <max_angle>0</max_angle>
+                        <samples>8</samples>
+                        <resolution>1</resolution>
+                        <min_angle>-0.296705972844</min_angle>  <!-- –17° in radians -->
+                        <max_angle> 0.052359877559</max_angle>  <!--  3° in radians -->
                     </vertical>
                 </scan>
                 <range>
-                    <min>0.08</min>
-                    <max>12.0</max>
+                    <min>0.10</min>
+                    <max>30.0</max>
                     <resolution>0.01</resolution>
                 </range>

File: src/avone/description/rgbdcamera.xacro (robot description, xacro)
@@ -13,9 +13,9 @@
     <child  link="rgbdcamera_link_optical"/>
     <!-- roll = -90°, pitch = 0, yaw = -90° -->
-    <origin xyz="0 0 0" rpy="0 0 0"/>
+    <origin xyz="0 0 0" rpy="${-pi/2} 0 ${-pi/2}"/>
   </joint>
   <link name="rgbdcamera_link_optical"/>
   <!-- 3) Gazebo ROS2 camera plugin on the OPTICAL link -->
-  <gazebo reference="rgbdcamera_link_optical">
+  <gazebo reference="rgbdcamera_link">
     <sensor name="rgbdcamera" type="rgbd">
       <topic>rgbdcamera</topic>
@@ -24,13 +24,19 @@
       <update_rate>30</update_rate>
       <camera>
-        <horizontal_fov>1.91986</horizontal_fov>
-        <image>
+        <horizontal_fov>1.212</horizontal_fov>
+         <image>
+          <width>640</width>
+          <height>480</height>
           <format>R8G8B8</format>
-          <width>1280</width>
-          <height>720</height>
         </image>
+        <!-- Depth image (640×480, L16) -->
+        <depth>
+          <width>640</width>
+          <height>480</height>
+          <format>L16</format>
+        </depth>
         <clip>
-          <near>0.3</near>
-          <far>20.0</far>
+          <near>0.1</near>
+          <far>10.0</far>
         </clip>
       </camera>

File: src/avone/description/robot.urdf.xacro (robot description, xacro)
@@ -7,4 +7,5 @@
     <!-- <xacro:include filename="depthcamera.xacro" /> -->
    <xacro:include filename="rgbdcamera.xacro" />
+    <!-- <xacro:include filename="dualrgbdcamera.xacro" /> -->
    <xacro:include filename="sensors.xacro" />
    <!-- <xacro:include filename="lidar.xacro" />  -->

Commit message: added waypoint hitting with nav2, can now drive round track

File: src/avone/description/camera.xacro (robot description, xacro)
@@ -30,13 +30,13 @@
             <camera>
             <camera_info_topic>camera/camera_info</camera_info_topic>
-                      <horizontal_fov>1.91986</horizontal_fov>
+                      <horizontal_fov>1.8</horizontal_fov>
                 <image>
                     <format>R8G8B8</format>
-                    <width>1280</width>
-                    <height>720</height>
+                           <width>640</width>
+          <height>360</height>
                 </image>
                 <clip>
                     <near>0.3</near>
-                    <far>20.0</far>
+                    <far>10.0</far>
                 </clip>
             </camera>

File: src/avone/description/depthcamera.xacro (robot description, xacro)
@@ -26,5 +26,5 @@
             <pose> 0 0 0 0 0 0 </pose>
             <visualize>true</visualize>
-            <update_rate>10</update_rate>
+            <update_rate>30</update_rate>
             <topic>depth/image_raw</topic>
             <camera>

File: src/avone/description/lidar.xacro (robot description, xacro)
@@ -4,5 +4,6 @@
         <parent link="chassis"/>
         <child link="laser_frame"/>
-        <origin xyz="2.4174 0 0.2977" rpy="0 0 0"/>
+         <origin xyz="2.3674 0 0.2977" rpy="0 -0.1 0"/>
+        <!-- <origin xyz="0.6909 0 0.772413" rpy="0 0.4 0"/> -->
     </joint>
     <link name="laser_frame">
@@ -39,5 +40,5 @@
                 <scan>
                     <horizontal>
-                        <samples>640</samples>
+                        <samples>1500</samples>
                         <resolution>1</resolution>
                         <min_angle>-1.8</min_angle>

File: src/avone/description/rgbdcamera.xacro (robot description, xacro)
@@ -24,7 +24,7 @@
       <update_rate>30</update_rate>
       <camera>
-        <horizontal_fov>1.212</horizontal_fov>
+        <horizontal_fov>1.8</horizontal_fov>
          <image>
-          <width>640</width>
+                <width>640</width>
           <height>480</height>
           <format>R8G8B8</format>
@@ -32,6 +32,6 @@
         <!-- Depth image (640×480, L16) -->
         <depth>
-          <width>640</width>
-          <height>480</height>
+           <width>640</width>
+          <height>360</height>
           <format>L16</format>
         </depth>

File: src/avone/description/robot.urdf.xacro (robot description, xacro)
@@ -4,9 +4,9 @@
     <xacro:include filename="ros2_control.xacro" />
     <xacro:include filename="gazebo_control.xacro"/>
-    <!-- <xacro:include filename="camera.xacro" />  -->
+    <xacro:include filename="camera.xacro" />
     <!-- <xacro:include filename="depthcamera.xacro" /> -->
    <xacro:include filename="rgbdcamera.xacro" />
     <!-- <xacro:include filename="dualrgbdcamera.xacro" /> -->
    <xacro:include filename="sensors.xacro" />
-   <!-- <xacro:include filename="lidar.xacro" />  -->
+   <xacro:include filename="lidar.xacro" />
 </robot>

Commit message: development on yolo model and implemented a cone landmark detection with the m8 3d lidar in conjunction with the cone pose estimate with yolo

File: src/avone/description/camera.xacro (robot description, xacro)
@@ -23,5 +23,5 @@
         <material>Gazebo/Red</material>
         <sensor name="camera" type="camera">
-            <gz_frame_id>camera_link</gz_frame_id>
+            <gz_frame_id>camera_link_optical</gz_frame_id>
             <pose> 0 0 0 0 0 0 </pose>
             <visualize>true</visualize>
@@ -30,5 +30,5 @@
             <camera>
             <camera_info_topic>camera/camera_info</camera_info_topic>
-                      <horizontal_fov>1.8</horizontal_fov>
+                      <horizontal_fov>1.2042771838760875</horizontal_fov>
                 <image>
                     <format>R8G8B8</format>
@@ -37,6 +37,6 @@
                 </image>
                 <clip>
-                    <near>0.3</near>
-                    <far>10.0</far>
+                    <near>0.1</near>
+                    <far>20.0</far>
                 </clip>
             </camera>

File: src/avone/description/depthcamera.xacro (robot description, xacro)
@@ -6,36 +6,33 @@
         <origin xyz="0.6909 0 0.772413" rpy="0 0 0"/>
     </joint>
-    <link name="depthcamera_link">
-        <visual>
-            <geometry>
-                <box size="0.010 0.03 0.03"/>
-            </geometry>
-            <material name="red"/>
-        </visual>
-    </link>
+    <link name="depthcamera_link"/>
     <joint name="depthcamera_optical_joint" type="fixed">
         <parent link="depthcamera_link"/>
         <child link="depthcamera_link_optical"/>
-        <origin xyz="0 0 0" rpy="0 0 0"/>
+        <origin xyz="0 0 0" rpy="${-pi/2} 0 ${-pi/2} "/>
+         <!-- <origin xyz="0 0 0" rpy="0 0 0"/> -->
     </joint>
-    <link name="depthcamera_link_optical"></link>
+    <link name="depthcamera_link_optical"/>
     <gazebo reference="depthcamera_link">
         <material>Gazebo/Red</material>
         <sensor name="depthcamera" type="depth">
+            <point_cloud>true</point_cloud>
             <gz_frame_id>depthcamera_link_optical</gz_frame_id>
+            <frame_id>depthcamera_link_optical</frame_id>
             <pose> 0 0 0 0 0 0 </pose>
             <visualize>true</visualize>
             <update_rate>30</update_rate>
             <topic>depth/image_raw</topic>
+            <camera_info_topic>depth/camera_info</camera_info_topic>
+            <always_on>1</always_on>
             <camera>
-                <horizontal_fov>1.089</horizontal_fov>
+                <horizontal_fov>1.2042771838760875</horizontal_fov>
                 <image>
-                    <format>R8G8B8</format>
                     <width>640</width>
-                    <height>480</height>
+                    <height>360</height>
                 </image>
                 <clip>
-                    <near>0.05</near>
-                    <far>8.0</far>
+                    <near>0.1</near>
+                    <far>6.0</far>
                 </clip>
             </camera>

File: src/avone/description/lidar.xacro (robot description, xacro)
@@ -4,5 +4,5 @@
         <parent link="chassis"/>
         <child link="laser_frame"/>
-         <origin xyz="2.3674 0 0.2977" rpy="0 -0.1 0"/>
+         <origin xyz="2.3674 0 0.2977" rpy="0 0 0"/>
         <!-- <origin xyz="0.6909 0 0.772413" rpy="0 0.4 0"/> -->
     </joint>
@@ -10,12 +10,5 @@
         <visual>
             <geometry>
-                <cylinder radius="0.025" length="0.04"/>
-            </geometry>
-            <material name="black"/>
-        </visual>
-        <visual>
-            <origin xyz="-0.125 0 -0.02"/>
-            <geometry>
-                <box size="0.3 0.05 0.01"/>
+                <cylinder radius="0.05" length="0.090"/>
             </geometry>
             <material name="black"/>
@@ -23,5 +16,5 @@
         <collision>
             <geometry>
-                <cylinder radius="0.05" length="0.04"/>
+                <cylinder radius="0.05" length="0.090"/>
             </geometry>
         </collision>
@@ -40,8 +33,8 @@
                 <scan>
                     <horizontal>
-                        <samples>1500</samples>
+                        <samples>2000</samples>
                         <resolution>1</resolution>
-                        <min_angle>-1.8</min_angle>
-                        <max_angle>1.8</max_angle>
+                        <min_angle>-1.3</min_angle>
+                        <max_angle>1.3</max_angle>
                     </horizontal>
                     <vertical>

File: src/avone/description/robot.urdf.xacro (robot description, xacro)
@@ -10,5 +10,5 @@
   <!-- 3) Simulation ros2_control -->
   <!-- <xacro:if value="$(arg use_sim)"> -->
-    <!-- <xacro:include filename="ros2_control.xacro"/> -->
+    <xacro:include filename="ros2_control.xacro"/>
     <!-- if you want gazebo_control in sim, uncomment this too -->
     <!-- <xacro:include filename="gazebo_control.xacro"/> -->
@@ -16,5 +16,5 @@
   <!-- 4) Real-hardware ros2_control -->
   <!-- <xacro:unless value="$(arg use_sim)"> -->
-    <xacro:include filename="ros2_control_hardware.xacro"/>
+    <!-- <xacro:include filename="ros2_control_hardware.xacro"/> -->
   <!-- </xacro:unless> -->
   <!-- 5) Sensors, cameras, lidar, etc. -->
@@ -23,3 +23,5 @@
   <xacro:include filename="sensors.xacro"/>
   <xacro:include filename="lidar.xacro"/>
+ <xacro:include filename="depthcamera.xacro"/>
+  <xacro:include filename="dualcamera.xacro"/>
 </robot>

File: src/avone/description/sensors.xacro (robot description, xacro)
@@ -23,5 +23,5 @@
     </joint>
   <link name="gps_antenna1_link">
-    <visual>
+    <!-- <visual>
       <geometry>
         <cylinder radius="0.0625" length="0.085"/>
@@ -33,5 +33,5 @@
         <cylinder radius="0.0625" length="0.085"/>
       </geometry>
-    </collision>
+    </collision> -->
   </link>
   <gazebo reference="gps_antenna1_link">
@@ -50,5 +50,5 @@
     </joint>
   <link name="gps_antenna2_link">
-    <visual>
+    <!-- <visual>
       <geometry>
         <cylinder radius="0.0625" length="0.085"/>
@@ -60,5 +60,5 @@
         <cylinder radius="0.0625" length="0.085"/>
       </geometry>
-    </collision>
+    </collision> -->
   </link>
   <gazebo reference="gps_antenna2_link">
