Commit message: avone package finalised, formatted and commented

File: src/avone/description/camera.xacro (robot description, xacro)
@@ -1,9 +1,27 @@
 <?xml version="1.0"?>
+<!--
+camera.xacro
+Purpose
+  Adds a simple simulated camera to the AV.ONE URDF for Gazebo.
+  Creates a physical mount frame (camera_link) and a REP-103 optical frame
+  (camera_link_optical), then attaches a Gazebo camera sensor.
+Frames
+  chassis -> camera_link -> camera_link_optical
+Topics
+  camera/image_raw
+  camera/camera_info
+Main tuning points
+  camera_joint origin: mount position and aim on the chassis
+  Gazebo sensor: update_rate, horizontal_fov, resolution, near/far clip
+-->
 <robot xmlns:xacro="http://www.ros.org/wiki/xacro" >
+    <!-- Fixed mount from chassis to the camera housing frame -->
     <joint name="camera_joint" type="fixed">
         <parent link="chassis"/>
         <child link="camera_link"/>
+        <!-- xyz in meters, rpy in radians -->
         <origin xyz="0.6909 0 0.772413" rpy="0 0 0"/>
     </joint>
+    <!-- Small visual box so the camera is visible in RViz and Gazebo -->
     <link name="camera_link">
         <visual>
@@ -14,4 +32,7 @@
         </visual>
     </link>
+    <!-- Optical frame for vision pipelines (REP-103 optical convention)
+         This rotation makes the optical frame axes match typical camera usage:
+           X right, Y down, Z forward -->
     <joint name="camera_optical_joint" type="fixed">
         <parent link="camera_link"/>
@@ -19,20 +40,26 @@
         <origin xyz="0 0 0" rpy="${-pi/2} 0 ${-pi/2}"/>
     </joint>
+    <!-- Optical frame link (no geometry, used for TF and frame_id) -->
     <link name="camera_link_optical"></link>
+    <!-- Gazebo sensor attached to camera_link, publishing using camera_link_optical -->
     <gazebo reference="camera_link">
         <material>Gazebo/Red</material>
         <sensor name="camera" type="camera">
+            <!-- Frame id that Gazebo will report for the image stream -->
             <gz_frame_id>camera_link_optical</gz_frame_id>
+            <!-- Pose relative to camera_link (leave zero if the joint origin is the mount) -->
             <pose> 0 0 0 0 0 0 </pose>
             <visualize>true</visualize>
             <update_rate>30</update_rate>
+            <!-- Image topic from the Gazebo camera sensor -->
             <topic>camera/image_raw</topic>
             <camera>
-            <camera_info_topic>camera/camera_info</camera_info_topic>
-                      <horizontal_fov>1.2042771838760875</horizontal_fov>
+                <camera_info_topic>camera/camera_info</camera_info_topic>
+                <!-- Horizontal FOV in radians -->
+                <horizontal_fov>1.2042771838760875</horizontal_fov>
                 <image>
                     <format>R8G8B8</format>
-                           <width>640</width>
-          <height>360</height>
+                    <width>640</width>
+                    <height>360</height>
                 </image>
                 <clip>

File: src/avone/description/lidar.xacro (robot description, xacro)
@@ -1,11 +1,29 @@
 <?xml version="1.0"?>
+<!--
+lidar.xacro
+Purpose
+  Defines a fixed mounted LiDAR link (laser_frame) on the chassis and attaches
+  a Gazebo gpu_lidar sensor that publishes a point cloud topic.
+Frames
+  chassis -> laser_frame
+Topics
+  lidar   (Gazebo sensor topic)
+Main tuning points
+  laser_joint origin: mount position and aim on the chassis
+  gpu_lidar scan: horizontal/vertical samples and FOV (min_angle/max_angle)
+  range: min/max and range resolution
+  update_rate: sensor publish frequency
+-->
 <robot xmlns:xacro="http://www.ros.org/wiki/xacro" >
+    <!-- Fixed mount from chassis to the LiDAR frame -->
     <joint name="laser_joint" type="fixed">
         <parent link="chassis"/>
         <child link="laser_frame"/>
-         <origin xyz="2.244 0 0.3464" rpy="0 0 0"/>
-        <!-- <origin xyz="0.6909 0 0.772413" rpy="0 0.4 0"/> -->
+        <!-- xyz in meters, rpy in radians -->
+        <origin xyz="2.244 0 0.3464" rpy="0 0 0"/>
     </joint>
+    <!-- LiDAR physical frame: visual + collision + inertial -->
     <link name="laser_frame">
+        <!-- Visual model used for viewing in RViz/Gazebo -->
         <visual>
             <geometry>
@@ -14,4 +32,5 @@
             <material name="black"/>
         </visual>
+        <!-- Collision geometry used by Gazebo physics -->
         <collision>
             <geometry>
@@ -19,17 +38,25 @@
             </geometry>
         </collision>
+        <!-- Inertial approximation (requires xacro:inertial_cylinder macro defined elsewhere) -->
         <xacro:inertial_cylinder mass="0.1" length="0.04" radius="0.05">
             <origin xyz="0 0 0" rpy="0 0 0"/>
         </xacro:inertial_cylinder>
     </link>
+    <!-- Gazebo sensor attached to laser_frame -->
     <gazebo reference="laser_frame">
         <material>Gazebo/Black</material>
+        <!-- GPU LiDAR: produces rays in a horizontal and vertical scan pattern -->
         <sensor name='gpu_lidar' type='gpu_lidar'>
+            <!-- Pose relative to the reference link; keep zero if laser_joint sets mount pose -->
             <pose relative_to='laser_frame'>0 0 0 0 0 0</pose>
+            <!-- Topic name published by Gazebo for this sensor -->
             <topic>lidar</topic>
-             <gz_frame_id>laser_frame</gz_frame_id>
+            <!-- Frame id stamped into the published messages -->
+            <gz_frame_id>laser_frame</gz_frame_id>
+            <!-- Publish frequency (Hz) -->
             <update_rate>10</update_rate>
             <ray>
                 <scan>
+                    <!-- Horizontal scan: 3600 samples across approx 149 degrees (±1.3 rad) -->
                     <horizontal>
                         <samples>3600</samples>
@@ -38,11 +65,15 @@
                         <max_angle>1.3</max_angle>
                     </horizontal>
+                    <!-- Vertical scan: 8 beams across about 20 degrees total -->
                     <vertical>
                         <samples>8</samples>
                         <resolution>1</resolution>
-                        <min_angle>-0.296705972844</min_angle>  <!-- –17° in radians -->
-                        <max_angle> 0.052359877559</max_angle>  <!--  3° in radians -->
+                        <!-- -17 degrees in radians -->
+                        <min_angle>-0.296705972844</min_angle>
+                        <!-- +3 degrees in radians -->
+                        <max_angle>0.052359877559</max_angle>
                     </vertical>
                 </scan>
+                <!-- Range limits and resolution -->
                 <range>
                     <min>0.10</min>
@@ -51,4 +82,5 @@
                 </range>
             </ray>
+            <!-- Sensor enable and visualization -->
             <always_on>1</always_on>
             <visualize>true</visualize>

File: src/avone/description/rgbdcamera.xacro (robot description, xacro)
@@ -1,39 +1,66 @@
 <?xml version="1.0"?>
+<!--
+rgbdcamera.xacro
+Purpose
+  Defines a fixed mounted RGBD camera on the chassis and adds a Gazebo RGBD
+  sensor that publishes both color and depth streams.
+Frames
+  chassis -> rgbdcamera_link -> rgbdcamera_link_optical
+Notes on optical frame
+  rgbdcamera_link_optical uses the REP-103/REP-105 optical convention:
+    X right, Y down, Z forward
+  The rpy of (-pi/2, 0, -pi/2) rotates a standard link frame into optical.
+Gazebo sensor
+  Uses a Gazebo 'rgbd' sensor (color + depth) with a single topic root.
+  Tune: update_rate, resolution, fov, clip near/far.
+Common gotchas
+  If you want the published messages stamped with the optical frame,
+  set gz_frame_id to rgbdcamera_link_optical (not rgbdcamera_link).
+-->
 <robot xmlns:xacro="http://www.ros.org/wiki/xacro">
-  <!-- 1) raw camera on the chassis -->
+  <!-- 1) Fixed mount from chassis to the camera body link -->
   <joint name="rgbdcamera_joint" type="fixed">
     <parent link="chassis"/>
     <child  link="rgbdcamera_link"/>
+    <!-- Mount pose (meters, radians) -->
     <origin xyz="0.6909 0 0.772413" rpy="0 0 0"/>
   </joint>
+  <!-- Camera body link (add visual/collision if you want to see it) -->
   <link name="rgbdcamera_link"/>
-  <!-- 2) optical frame, with X→right, Y→down, Z→forward -->
+  <!-- 2) Optical frame: X right, Y down, Z forward -->
   <joint name="rgbdcamera_optical_joint" type="fixed">
     <parent link="rgbdcamera_link"/>
     <child  link="rgbdcamera_link_optical"/>
-    <!-- roll = -90°, pitch = 0, yaw = -90° -->
+    <!-- roll=-90°, yaw=-90°: standard optical frame rotation -->
     <origin xyz="0 0 0" rpy="${-pi/2} 0 ${-pi/2}"/>
   </joint>
   <link name="rgbdcamera_link_optical"/>
-  <!-- 3) Gazebo ROS2 camera plugin on the OPTICAL link -->
+  <!-- 3) Gazebo RGBD sensor attached to the camera link -->
   <gazebo reference="rgbdcamera_link">
     <sensor name="rgbdcamera" type="rgbd">
+      <!-- Topic namespace/root for this sensor -->
       <topic>rgbdcamera</topic>
+      <!-- Frame id stamped into Gazebo-published messages -->
+      <!-- Consider switching this to rgbdcamera_link_optical if you want optical stamping -->
       <gz_frame_id>rgbdcamera_link</gz_frame_id>
+      <!-- Keep zero if mounting is already defined by the joint -->
       <pose>0 0 0 0 0 0</pose>
+      <!-- Publish rate (Hz) -->
       <update_rate>30</update_rate>
       <camera>
         <horizontal_fov>1.2042771838760875</horizontal_fov>
-         <image>
-                <width>640</width>
+        <!-- Color image stream -->
+        <image>
+          <width>640</width>
           <height>360</height>
           <format>R8G8B8</format>
         </image>
-        <!-- Depth image (640×480, L16) -->
+        <!-- Depth image stream -->
         <depth>
-           <width>640</width>
+          <width>640</width>
           <height>360</height>
           <format>L16</format>
         </depth>
+        <!-- Clipping planes -->
         <clip>
           <near>0.1</near>

File: src/avone/description/robot.urdf.xacro (robot description, xacro)
@@ -1,16 +1,19 @@
 <?xml version="1.0"?>
 <robot xmlns:xacro="http://www.ros.org/wiki/xacro" name="robot">
-  <!-- 2) Core links/visuals etc -->
+  <!-- ========================================================= -->
+  <!-- Robot top-level URDF (robot.urdf.xacro)                    -->
+  <!-- ========================================================= -->
+  <!-- This file composes the robot from smaller xacro parts.     -->
+  <!-- Core vehicle kinematic tree + visuals + collisions -->
   <xacro:include filename="robot_core.xacro"/>
+  <!-- Control interface -->
   <!-- FOR SIMULATION -->
-  <!-- <xacro:include filename="ros2_control.xacro"/> -->
+  <xacro:include filename="ros2_control.xacro"/>
   <!-- FOR REAL HARDWARE -->
-  <xacro:include filename="ros2_control_hardware.xacro"/>
-  <!-- 5) Sensors, cameras, lidar, etc. -->
+  <!-- <xacro:include filename="ros2_control_hardware.xacro"/> -->
+ <!-- Sensors, cameras, lidar, etc. -->
   <xacro:include filename="camera.xacro"/>
   <xacro:include filename="rgbdcamera.xacro"/>
   <xacro:include filename="sensors.xacro"/>
   <xacro:include filename="lidar.xacro"/>
- <!-- <xacro:include filename="depthcamera.xacro"/>  -->
-  <!-- <xacro:include filename="dualcamera.xacro"/>  -->
 </robot>
