Commit message: avone package finalised, formatted and commented

File: src/avone/description/robot_core.xacro (robot description, xacro)
@@ -1,60 +1,101 @@
 <?xml version="1.0"?>
-<robot xmlns:xacro="http://www.ros.org/wiki/xacro" >
-    <xacro:include filename="inertial_macros.xacro"/>
-    <!-- FOR GAZEBO SIM - CHANGE MESH TO FULL PATH - EG: -->
-    <!-- Replace package:// with file:///home/avone/avone_ws/src/ (user and folder dependant)-->
-    <!-- <mesh filename="file:///home/avone/avone_ws/src/avone/description/assets/chassis.stl"/> -->
-    <material name="white">
-        <color rgba="1 1 1 1" />
-    </material>
-    <material name="orange">
-        <color rgba="1 0.3 0.1 1"/>
-    </material>
-    <material name="blue">
-        <color rgba="0.2 0.2 1 1"/>
-    </material>
-    <material name="black">
-        <color rgba="0 0 0 1"/>
-    </material>
-   <!-- BASE LINK -->
-    <!-- BASE LINK -->
-    <link name="base_link">
-      <!-- You can add visual, collision, and inertial info here -->
-    </link>
-    <joint name="base_footprint_joint" type="fixed">
-        <parent link="base_link"/>
-        <child link="base_footprint"/>
-        <origin xyz="1.0 0 0" rpy="0 0 0"/>
-    </joint>
-    <link name="base_footprint">
-    </link>
-    <!-- Fixed joint connecting base_link to chassis -->
-    <joint name="base_to_chassis" type="fixed">
-      <parent link="base_link"/>
-      <child link="chassis"/>
-      <origin xyz="0 0 0.2028" rpy="0 0 0"/>
-    </joint>
-    <link name="chassis">
-        <visual>
-            <origin xyz="2.2924 -0.00985747 0.0751" rpy="3.14159 0 1.5708"/>
-            <geometry>
-                  <mesh filename="package://avone/description/assets/chassis.stl"/>
-            </geometry>
-            <material name="blue"/>
-        </visual>
-        <collision>
-            <origin xyz="2.2924 -0.00985747 0.0751" rpy="3.14159 0 1.5708"/>
-            <geometry>
-                    <mesh filename="package://avone/description/assets/chassis.stl"/>
-            </geometry>
-        </collision>
-        <xacro:inertial_box mass="152" x="2.4" y="0.67" z="0.5">
-            <origin xyz="0.812063 -0.000266118 0.127823" rpy="0 0 0"/>
-        </xacro:inertial_box>
-     <!-- Part rear_suspension -->
+<robot xmlns:xacro="http://www.ros.org/wiki/xacro">
+  <!-- ========================================================= -->
+  <!-- AV.ONE Robot Core Model (robot_core.xacro)                 -->
+  <!-- ========================================================= -->
+  <!-- Purpose:
+       - Defines the main kinematic tree (links + joints)
+       - Adds visual + collision geometry (meshes)
+       - Provides inertial approximations via inertial macros
+       - Acts as the base include for sensors/controllers xacros
+       Notes:
+       - Mesh paths are hard-coded to a local workspace path for Gazebo.
+         If you move machines/users, update the file:///home/... paths.
+       - This file defines the vehicle body, wheels, and steering joints.
+       - Gazebo plugin blocks at the end are currently disabled via XML comments.
+  -->
+  <!-- ========================================================= -->
+  <!-- Includes                                                   -->
+  <!-- ========================================================= -->
+  <xacro:include filename="inertial_macros.xacro"/>
+  <!-- ========================================================= -->
+  <!-- Mesh path notes                                             -->
+  <!-- ========================================================= -->
+  <!-- Could not figure out a way to have meshes work for both gazebo simulator and rviz  -->
+  <!-- without hard-coding path. Using package is ideal way, but doesnt work with gazebo. -->
+  <!-- Default (recommended): use package:// so it works on any machine -->
+  <!-- Example: <mesh filename="package://avone/description/assets/chassis.stl"/> -->
+  <!-- Gazebo / sim fallback: if your simulator does NOT resolve package:// URIs,
+       swap package://avone/description/assets/... with an absolute file:// path.
+       Example:
+       <mesh filename="file:///home/avone/avone_ws/src/avone/description/assets/chassis.stl"/> -->
+  <!-- ========================================================= -->
+  <!-- Materials                                                   -->
+  <!-- ========================================================= -->
+  <material name="white">
+    <color rgba="1 1 1 1"/>
+  </material>
+  <material name="orange">
+    <color rgba="1 0.3 0.1 1"/>
+  </material>
+  <material name="blue">
+    <color rgba="0.2 0.2 1 1"/>
+  </material>
+  <material name="black">
+    <color rgba="0 0 0 1"/>
+  </material>
+  <!-- ========================================================= -->
+  <!-- Base frames                                                 -->
+  <!-- ========================================================= -->
+  <!-- base_link: primary robot base frame (REP-103 style root) -->
+  <link name="base_link">
+    <!-- You can add visual, collision, and inertial info here -->
+  </link>
+  <!-- base_footprint: typically planar reference for navigation -->
+  <joint name="base_footprint_joint" type="fixed">
+    <parent link="base_link"/>
+    <child link="base_footprint"/>
+    <origin xyz="1.0 0 0" rpy="0 0 0"/>
+  </joint>
+  <link name="base_footprint"/>
+  <!-- ========================================================= -->
+  <!-- Chassis connection                                          -->
+  <!-- ========================================================= -->
+  <!-- Fixed joint connecting base_link to chassis -->
+  <joint name="base_to_chassis" type="fixed">
+    <parent link="base_link"/>
+    <child link="chassis"/>
+    <origin xyz="0 0 0.2028" rpy="0 0 0"/>
+  </joint>
+  <!-- ========================================================= -->
+  <!-- Chassis link                                                 -->
+  <!-- ========================================================= -->
+  <link name="chassis">
+    <!-- Main chassis body mesh -->
+    <visual>
+      <origin xyz="2.2924 -0.00985747 0.0751" rpy="3.14159 0 1.5708"/>
+      <geometry>
+        <mesh filename="file:///home/avone/avone_ws/src/avone/description/assets/chassis.stl"/>
+      </geometry>
+      <material name="blue"/>
+    </visual>
+    <collision>
+      <origin xyz="2.2924 -0.00985747 0.0751" rpy="3.14159 0 1.5708"/>
+      <geometry>
+        <mesh filename="file:///home/avone/avone_ws/src/avone/description/assets/chassis.stl"/>
+      </geometry>
+    </collision>
+    <!-- Approx inertial model for chassis -->
+    <xacro:inertial_box mass="152" x="2.4" y="0.67" z="0.5">
+      <origin xyz="0.812063 -0.000266118 0.127823" rpy="0 0 0"/>
+    </xacro:inertial_box>
+    <!-- ===================================================== -->
+    <!-- Rear suspension meshes                                  -->
+    <!-- ===================================================== -->
+    <!-- Part rear_suspension -->
     <visual>
       <origin xyz="-0.170629 -0.28192 0.105" rpy="3.14159 5.47382e-48 -0.0851102"/>
       <geometry>
-        <mesh filename="package://avone/description/assets/rear_suspension.stl"/>
+        <mesh filename="file:///home/avone/avone_ws/src/avone/description/assets/rear_suspension.stl"/>
       </geometry>
       <material name="blue"/>
@@ -63,5 +104,5 @@
       <origin xyz="-0.170629 -0.28192 0.105" rpy="3.14159 5.47382e-48 -0.0851102"/>
       <geometry>
-        <mesh filename="package://avone/description/assets/rear_suspension.stl"/>
+        <mesh filename="file:///home/avone/avone_ws/src/avone/description/assets/rear_suspension.stl"/>
       </geometry>
     </collision>
@@ -70,5 +111,5 @@
       <origin xyz="0.189017 0.312761 0.105" rpy="-3.14159 2.33363e-61 -3.05648"/>
       <geometry>
-        <mesh filename="package://avone/description/assets/rear_suspension.stl"/>
+        <mesh filename="file:///home/avone/avone_ws/src/avone/description/assets/rear_suspension.stl"/>
       </geometry>
       <material name="blue"/>
@@ -77,12 +118,15 @@
       <origin xyz="0.189017 0.312761 0.105" rpy="-3.14159 2.33363e-61 -3.05648"/>
       <geometry>
-        <mesh filename="package://avone/description/assets/rear_suspension.stl"/>
-      </geometry>
-    </collision>
+        <mesh filename="file:///home/avone/avone_ws/src/avone/description/assets/rear_suspension.stl"/>
+      </geometry>
+    </collision>
+    <!-- ===================================================== -->
+    <!-- Front suspension meshes                                 -->
+    <!-- ===================================================== -->
     <!-- Part front_suspension -->
     <visual>
       <origin xyz="1.6032 0.2935 0.075" rpy="3.14159 -1.54112e-16 1.5708"/>
       <geometry>
-        <mesh filename="package://avone/description/assets/front_suspension.stl"/>
+        <mesh filename="file:///home/avone/avone_ws/src/avone/description/assets/front_suspension.stl"/>
       </geometry>
       <material name="blue"/>
@@ -91,5 +135,5 @@
       <origin xyz="1.6032 0.2935 0.075" rpy="3.14159 -1.54112e-16 1.5708"/>
       <geometry>
-        <mesh filename="package://avone/description/assets/front_suspension.stl"/>
+        <mesh filename="file:///home/avone/avone_ws/src/avone/description/assets/front_suspension.stl"/>
       </geometry>
     </collision>
@@ -98,5 +142,5 @@
       <origin xyz="1.8748 -0.2935 0.075" rpy="-3.14159 1.54112e-16 -1.5708"/>
       <geometry>
-        <mesh filename="package://avone/description/assets/front_suspension.stl"/>
+        <mesh filename="file:///home/avone/avone_ws/src/avone/description/assets/front_suspension.stl"/>
       </geometry>
       <material name="blue"/>
@@ -105,12 +149,15 @@
       <origin xyz="1.8748 -0.2935 0.075" rpy="-3.14159 1.54112e-16 -1.5708"/>
       <geometry>
-        <mesh filename="package://avone/description/assets/front_suspension.stl"/>
-      </geometry>
-    </collision>
-  <!-- REAR WHEEL HUB LEFT -->
+        <mesh filename="file:///home/avone/avone_ws/src/avone/description/assets/front_suspension.stl"/>
+      </geometry>
+    </collision>
+    <!-- ===================================================== -->
+    <!-- Rear wheel hub meshes (cosmetic on chassis link)         -->
+    <!-- ===================================================== -->
+    <!-- REAR WHEEL HUB LEFT -->
     <visual>
       <origin xyz="-0.181377 0.297001 -0.105" rpy="6.30462e-15 0 -6.18615e-05"/>
       <geometry>
-        <mesh filename="package://avone/description/assets/rear_wheel_hub.stl"/>
+        <mesh filename="file:///home/avone/avone_ws/src/avone/description/assets/rear_wheel_hub.stl"/>
       </geometry>
       <material name="white"/>
@@ -119,12 +166,12 @@
       <origin xyz="-0.181377 0.297001 -0.105" rpy="6.30462e-15 0 -6.18615e-05"/>
       <geometry>
-        <mesh filename="package://avone/description/assets/rear_wheel_hub.stl"/>
-      </geometry>
-    </collision>
-  <!-- REAR WHEEL HUB RIGHT -->
+        <mesh filename="file:///home/avone/avone_ws/src/avone/description/assets/rear_wheel_hub.stl"/>
+      </geometry>
+    </collision>
+    <!-- REAR WHEEL HUB RIGHT -->
     <visual>
       <origin xyz="0.181423 -0.296978 -0.105" rpy="3.10966e-15 7.00787e-15 -3.14153"/>
       <geometry>
-        <mesh filename="package://avone/description/assets/rear_wheel_hub.stl"/>
+        <mesh filename="file:///home/avone/avone_ws/src/avone/description/assets/rear_wheel_hub.stl"/>
       </geometry>
       <material name="white"/>
@@ -133,258 +180,245 @@
       <origin xyz="0.181423 -0.296978 -0.105" rpy="3.10966e-15 7.00787e-15 -3.14153"/>
       <geometry>
-        <mesh filename="package://avone/description/assets/rear_wheel_hub.stl"/>
-      </geometry>
-    </collision>
-  </link>
+        <mesh filename="file:///home/avone/avone_ws/src/avone/description/assets/rear_wheel_hub.stl"/>
+      </geometry>
+    </collision>
+  </link>
+  <!-- ========================================================= -->
+  <!-- Gazebo material override for chassis                        -->
+  <!-- ========================================================= -->
   <gazebo reference="chassis">
     <material>Gazebo/Blue</material>
   </gazebo>
-    <!-- LEFT WHEEL LINK (RLMotor) -->
-    <joint name="RLMotor" type="continuous">
-        <origin xyz="4.71381e-05 0.693977 3.30291e-15" rpy="1.5708 0 -6.18615e-05"/>
-        <parent link="chassis"/>
-        <child link="left_motor"/>
-        <axis xyz="0 0 -1"/>
-     <dynamics damping="0.02" friction="0.2"/>
-      <limit
-          effort="108.6"
-          velocity="36.65"/>
-          <!-- NEED TO FIND THIS ^^ -->
-        <!--
-            effort (Nm) = kT × I_cont
-              ≈ 0.955 Nm/A × 95 A = 91 Nm
-            velocity (rad/s) = Kv × V
-              ≈ (10 rpm/V × 96 V) × (2π/60) ≈ 100.7 rad/s
-            :contentReference[oaicite:0]{index=0}
-        -->
-      </joint>
-    <link name="left_motor">
-        <visual>
-            <origin xyz="-8.09391e-17 7.65875e-18 0.17" rpy="1.5708 0 0"/>
-            <geometry>
-                    <mesh filename="package://avone/description/assets/wheel.stl"/>
-                 <!--  <box size="0.3 0.3 0.15"/> -->
-            </geometry>
-            <material name="black"/>
-        </visual>
-        <collision>
-            <origin xyz="-8.09391e-17 7.65875e-18 0.17" rpy="1.5708 0 0"/>
-            <geometry>
-                     <!--<mesh filename="package://avone/description/assets/wheel.stl"/>    -->
-                                        <sphere radius="0.203"/>
-                 <!--  <box size="0.3 0.3 0.15"/> -->
-            </geometry>
-        </collision>
-        <xacro:inertial_cylinder mass="9.8" length="0.2" radius="0.2">
-            <origin xyz="-8.09407e-17 -1.33567e-17 0.0496398" rpy="0 0 0"/>
-        </xacro:inertial_cylinder>
-    </link>
-    <gazebo reference="left_motor">
-        <material>Gazebo/Grey</material>
-    </gazebo>
-    <!-- RIGHT WHEEL LINK (RRMotor) -->
-    <joint name="RRMotor" type="continuous">
-        <origin xyz="4.71381e-05 -0.693977 2.30371e-15" rpy="1.5708 0 -3.14153"/>
-        <parent link="chassis"/>
-        <child link="right_motor"/>
-        <axis xyz="0 0 1"/>
-      <dynamics damping="0.02" friction="0.2"/>
-      <limit
-          effort="108.6"
-          velocity="36.65"/>
-    </joint>
-    <link name="right_motor">
-        <visual>
-            <origin xyz="-1.59877e-17 7.65404e-18 0.17" rpy="1.5708 0 0"/>
-            <geometry>
-                    <mesh filename="package://avone/description/assets/wheel.stl"/>
-                 <!--  <box size="0.3 0.3 0.15"/> -->
-            </geometry>
-            <material name="black"/>
-        </visual>
-        <collision>
-            <origin xyz="-1.59877e-17 7.65404e-18 0.17" rpy="1.5708 0 0"/>
-            <geometry>
-                     <sphere radius="0.203"/>
-                 <!--  <box size="0.3 0.3 0.15"/> -->
-            </geometry>
-        </collision>
-        <xacro:inertial_cylinder mass="9.8" length="0.2" radius="0.2">
-            <origin xyz="-1.66794e-17 -1.33614e-17 0.0496398" rpy="0 0 0"/>
-        </xacro:inertial_cylinder>
-    </link>
-    <gazebo reference="right_motor">
-        <material>Gazebo/Grey</material>
-    </gazebo>
-    <!-- FRONT RIGHT STEERING ASSEMBLY -->
-    <!-- FRONT RIGHT STEERING ASSEMBLY -->
-    <joint name="RSteer" type="revolute">
-        <origin xyz="1.739 -0.584139 0.075" rpy="-3.14159 0 -1.5708"/>
-        <parent link="chassis"/>
-        <child link="front_right_wheel_hub"/>
-        <axis xyz="0 0 -1"/>
-        <limit  effort="33.4"
-          velocity="1.0"
-          lower="-0.610865"
-          upper="0.610865"/>
-          <dynamics damping="0.1" friction="0.05"/>
-    </joint>
-    <link name="front_right_wheel_hub">
-        <visual>
-            <origin xyz="-0.290639 0.1358 0.18" rpy="-3.14159 0 0"/>
-            <geometry>
-                    <mesh filename="package://avone/description/assets/front_wheel_hub.stl"/>
-                 <!--  <box size="0.3 0.3 0.15"/> -->
-            </geometry>
-            <material name="white"/>
-        </visual>
-        <collision>
-            <origin xyz="-0.290639 0.1358 0.18" rpy="-3.14159 0 0"/>
-            <geometry>
-                    <mesh filename="package://avone/description/assets/front_wheel_hub.stl"/>
-                 <!--  <box size="0.3 0.3 0.15"/> -->
-            </geometry>
-        </collision>
-        <xacro:inertial_box mass="1.6" x="0.1" y="0.1" z="0.1">
-            <origin xyz="0.0824722 0 0.09" rpy="0 0 0"/>
-        </xacro:inertial_box>
-    </link>
-    <gazebo reference="front_right_wheel_hub">
-        <material>Gazebo/Black</material>
-    </gazebo>
-    <joint name="FRWheel" type="continuous">
-        <origin xyz="0.10836 0 0.09" rpy="1.5708 0 -1.5708"/>
-        <parent link="front_right_wheel_hub"/>
-        <child link="front_right_wheel"/>
-        <axis xyz="0 0 1"/>
-        <limit effort="50" velocity="100"/>
-        <dynamics damping="0.0" friction="0.0"/>
-    </joint>
-    <link name="front_right_wheel">
-        <visual>
-            <origin xyz="2.22045e-16 0 0.17" rpy="1.5708 0 1.5708"/>
-            <geometry>
-                    <mesh filename="package://avone/description/assets/wheel.stl"/>
-                 <!--  <box size="0.3 0.3 0.15"/> -->
-            </geometry>
-            <material name="black"/>
-        </visual>
-        <collision>
-            <origin xyz="2.22045e-16 0 0.17" rpy="1.5708 0 1.5708"/>
-            <geometry>
-                   <!--<mesh filename="package://avone/description/assets/wheel.stl"/>    -->
-                                        <sphere radius="0.203"/>
-                 <!--  <box size="0.3 0.3 0.15"/> -->
-            </geometry>
-        </collision>
-        <xacro:inertial_cylinder mass="9.8" length="0.2" radius="0.2">
-            <origin xyz="2.33038e-16 0 0.0496398" rpy="0 0 0"/>
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
File: src/avone/description/ros2_control.xacro (robot description, xacro)
@@ -1,4 +1,31 @@
 <?xml version="1.0"?>
 <robot xmlns:xacro="http://www.ros.org/wiki/xacro">
+<!-- ========================================================= -->
+<!-- AV.ONE ros2_control (SIMULATION / GAZEBO)                   -->
+<!-- File: ros2_control.xacro                                    -->
+<!-- ========================================================= -->
+<!-- Purpose:
+     - Defines the ros2_control "system" used in Gazebo simulation.
+     - Uses the GazeboSimSystem hardware plugin (gz_ros2_control) so Gazebo
+       provides joint states and accepts joint commands via ros2_control.
+     - Loads the Gazebo ROS 2 Control plugin that connects Gazebo to
+       controller_manager and reads the controller YAML.
+     What this file contains:
+     1) <ros2_control name="GazeboSimSystem" type="system">
+          <hardware>
+            <plugin>gz_ros2_control/GazeboSimSystem</plugin>
+          </hardware>
+        - Joint interface declarations:
+            LSteer, RSteer: position command + position state
+            RLMotor, RRMotor: velocity command + velocity + position state
+            FLWheel, FRWheel: position state only
+     2) <gazebo> plugin block:
+        - gz_ros2_control::GazeboSimROS2ControlPlugin
+        - Reads robot_description from robot_state_publisher
+        - Loads controller parameters from:
+            $(find avone)/config/ackermann_drive_controller.yaml
+     How it is used:
+     - Included by robot.urdf.xacro when running in Gazebo.
+     - For real hardware you normally include ros2_control_hardware.xacro instead. -->
   <ros2_control name="GazeboSimSystem" type="system">
     <hardware>

File: src/avone/description/ros2_control_hardware.xacro (robot description, xacro)
@@ -1,19 +1,51 @@
 <?xml version="1.0"?>
 <robot xmlns:xacro="http://www.ros.org/wiki/xacro">
+<!-- ========================================================= -->
+<!-- AV.ONE ros2_control (HARDWARE)                             -->
+<!-- File: ros2_control_hardware.xacro                          -->
+<!-- ========================================================= -->
+<!-- Purpose:
+     - Defines the ros2_control "system" for REAL hardware.
+     - Loads the AvoneSystemHardware plugin and exposes steering + drive joints.
+     - Provides CAN IDs and limits as parameters to the hardware plugin.
+     What this file contains:
+     - <ros2_control ... type="system"> block
+     - <hardware><plugin>avone/AvoneSystemHardware</plugin> + <param> list
+     - Joint interface declarations:
+         LSteer, RSteer: position command + position state
+         RLMotor, RRMotor: velocity command + velocity + position state
+         FLWheel, FRWheel: position state only
+     How it is used:
+     - Included by robot.urdf.xacro when running on the real car.
+     - In simulation you normally include ros2_control.xacro instead.
+-->
   <ros2_control name="AVONE_ros2_control" type="system">
     <hardware>
       <plugin>avone/AvoneSystemHardware</plugin>
-      <!-- Your existing params -->
+      <!-- Maximum allowed steering angle in radians (soft limit for steering commands and safety clamping) -->
       <param name="max_steer_angle">0.610865</param>
+      <!-- Minimum allowed steering angle in radians (negative direction limit for steering commands and safety clamping) -->
       <param name="min_steer_angle">-0.610865</param>
+      <!-- Maximum rear motor speed in RPM used as a limit when converting commands or clamping outputs -->
       <param name="max_rpm">300</param>
+      <!-- If true, do not open CAN or transmit real frames; simulate joint states from commands instead -->
+      <param name="sim_mode">false</param>
+      <!-- Linux SocketCAN interface name to bind to, e.g. can0 for real bus or vcan0 for virtual testing -->
       <param name="can_interface">can0</param>
+      <!-- CAN bus bitrate   -->
       <param name="can_baudrate">250000</param>
+      <!-- Read timeout in milliseconds for polling CAN receive  -->
       <param name="read_timeout_ms">20</param>
+      <!-- CAN ID for left motor rpm-->
       <param name="l_motor_can_id">0x8CF11E05</param>
+      <!-- CAN ID for rights motor rpm-->
       <param name="r_motor_can_id">0x8CF11E06</param>
+      <!-- CAN ID for steering angle reading-->
       <param name="steer_can_id">0x0D</param>
+      <!-- CAN ID that this interface transmits left motor speed commands on  -->
       <param name="cmd_l_motor_can_id">0x0B</param>
+      <!-- CAN ID that this interface transmits right motor speed commands on ( -->
       <param name="cmd_r_motor_can_id">0x0A</param>
+      <!-- CAN ID that this interface transmits steering commands on -->
       <param name="cmd_steer_can_id">0x09</param>
     </hardware>
