Commit message: Initial commit with entire ros workspace, including cone detection, position estimation

File: src/avone/description/robot.urdf.xacro (robot description, xacro)
@@ -2,3 +2,10 @@
 <robot xmlns:xacro="http://www.ros.org/wiki/xacro"  name="robot">
     <xacro:include filename="robot_core.xacro" />
+    <xacro:include filename="ros2_control.xacro" />
+    <xacro:include filename="gazebo_control.xacro"/>
+    <xacro:include filename="camera.xacro" />
+    <!--<xacro:include filename="depthcamera.xacro" /> -->
+  <!-- <xacro:include filename="rgbdcamera.xacro" /> -->
+   <xacro:include filename="sensors.xacro" />
+   <xacro:include filename="lidar.xacro" />
 </robot>

File: src/avone/description/robot_core.xacro (robot description, xacro)
@@ -1,323 +1,368 @@
 <?xml version="1.0"?>
-<robot xmlns:xacro="http://www.ros.org/wiki/xacro" name="avone">
-  <!-- Base Link (new root) -->
-  <link name="base_link"/>
-  <!-- Joint connecting base_link to chassis_suspension -->
-  <joint name="base_to_chassis_joint" type="fixed">
-    <parent link="base_link"/>
-    <child link="chassis_suspension"/>
-    <origin xyz="-0.1706 0 -0.105" rpy="0 0 0"/>
-  </joint>
-  <!-- Existing chassis_suspension link (previous root) -->
-  <link name="chassis_suspension">
-    <inertial>
-      <origin xyz="0.812063 -0.000266118 0.127823" rpy="0 0 0"/>
-      <mass value="152"/>
-      <inertia ixx="16.787" ixy="-0.0144134" ixz="2.17886" iyy="94.5857" iyz="0.0189829" izz="101.287"/>
-    </inertial>
-    <!-- Part rear_wheel_hub -->
-    <visual>
-      <origin xyz="-0.181377 0.297001 -0.105" rpy="6.30462e-15 -0 -6.18615e-05"/>
-      <geometry>
-        <mesh filename="package://avone/avonemodel/assets/rear_wheel_hub.stl"/>
-      </geometry>
-      <material name="rear_wheel_hub_material">
-        <color rgba="0.972549 0.529412 0.00392157 1.0"/>
-      </material>
-    </visual>
-    <collision>
-      <origin xyz="-0.181377 0.297001 -0.105" rpy="6.30462e-15 -0 -6.18615e-05"/>
-      <geometry>
-        <mesh filename="package://avone/avonemodel/assets/rear_wheel_hub.stl"/>
-      </geometry>
-    </collision>
-    <!-- Part rear_wheel_hub_2 -->
+<robot xmlns:xacro="http://www.ros.org/wiki/xacro" >
+    <xacro:include filename="inertial_macros.xacro"/>
+    <material name="white">
+        <color rgba="1 1 1 1" />
+    </material>
+    <material name="orange">
+        <color rgba="1 0.3 0.1 1"/>
+    </material>
+    <material name="blue">
+        <color rgba="0.2 0.2 1 1"/>
+    </material>
+    <material name="black">
+        <color rgba="0 0 0 1"/>
+    </material>
+   <!-- BASE LINK -->
+    <!-- BASE LINK -->
+    <link name="base_link">
+      <!-- You can add visual, collision, and inertial info here -->
+    </link>
+    <joint name="base_footprint_joint" type="fixed">
+        <parent link="base_link"/>
+        <child link="base_footprint"/>
+        <origin xyz="0 0 0" rpy="0 0 0"/>
+    </joint>
+    <link name="base_footprint">
+    </link>
+    <!-- Fixed joint connecting base_link to chassis -->
+    <joint name="base_to_chassis" type="fixed">
+      <parent link="base_link"/>
+      <child link="chassis"/>
+      <origin xyz="0 0 0.2028" rpy="0 0 0"/>
+    </joint>
+    <link name="chassis">
+        <visual>
+            <origin xyz="2.2924 -0.00985747 0.0751" rpy="3.14159 0 1.5708"/>
+            <geometry>
+                  <mesh filename="file:///home/jay/ros2_ws/src/avone/description/assets/chassis.stl"/>
+                 <!-- <mesh filename="package://avone/description/assets/chassis.stl"/> -->
+                 <!--  <box size="0.3 0.3 0.15"/> -->
+            </geometry>
+            <material name="blue"/>
+        </visual>
+        <collision>
+            <origin xyz="2.2924 -0.00985747 0.0751" rpy="3.14159 0 1.5708"/>
+            <geometry>
+                    <mesh filename="file:///home/jay/ros2_ws/src/avone/description/assets/chassis.stl"/>
+                 <!--  <box size="0.3 0.3 0.15"/> -->
+            </geometry>
+        </collision>
+        <xacro:inertial_box mass="152" x="2.4" y="0.67" z="0.5">
+            <origin xyz="0.812063 -0.000266118 0.127823" rpy="0 0 0"/>
+        </xacro:inertial_box>
+     <!-- Part rear_suspension -->
+    <visual>
+      <origin xyz="-0.170629 -0.28192 0.105" rpy="3.14159 5.47382e-48 -0.0851102"/>
+      <geometry>
+        <mesh filename="file:///home/jay/ros2_ws/src/avone/description/assets/rear_suspension.stl"/>
+      </geometry>
+      <material name="blue"/>
+    </visual>
+    <collision>
+      <origin xyz="-0.170629 -0.28192 0.105" rpy="3.14159 5.47382e-48 -0.0851102"/>
+      <geometry>
+        <mesh filename="file:///home/jay/ros2_ws/src/avone/description/assets/rear_suspension.stl"/>
+      </geometry>
+    </collision>
+    <!-- Part rear_suspension_2 -->
+    <visual>
+      <origin xyz="0.189017 0.312761 0.105" rpy="-3.14159 2.33363e-61 -3.05648"/>
+      <geometry>
+        <mesh filename="file:///home/jay/ros2_ws/src/avone/description/assets/rear_suspension.stl"/>
+      </geometry>
+      <material name="blue"/>
+    </visual>
+    <collision>
+      <origin xyz="0.189017 0.312761 0.105" rpy="-3.14159 2.33363e-61 -3.05648"/>
+      <geometry>
+        <mesh filename="file:///home/jay/ros2_ws/src/avone/description/assets/rear_suspension.stl"/>
+      </geometry>
+    </collision>
+    <!-- Part front_suspension -->
+    <visual>
+      <origin xyz="1.6032 0.2935 0.075" rpy="3.14159 -1.54112e-16 1.5708"/>
+      <geometry>
+        <mesh filename="file:///home/jay/ros2_ws/src/avone/description/assets/front_suspension.stl"/>
+      </geometry>
+      <material name="blue"/>
+    </visual>
+    <collision>
+      <origin xyz="1.6032 0.2935 0.075" rpy="3.14159 -1.54112e-16 1.5708"/>
+      <geometry>
+        <mesh filename="file:///home/jay/ros2_ws/src/avone/description/assets/front_suspension.stl"/>
+      </geometry>
+    </collision>
+    <!-- Part front_suspension_2 -->
+    <visual>
+      <origin xyz="1.8748 -0.2935 0.075" rpy="-3.14159 1.54112e-16 -1.5708"/>
+      <geometry>
+        <mesh filename="file:///home/jay/ros2_ws/src/avone/description/assets/front_suspension.stl"/>
+      </geometry>
+      <material name="blue"/>
+    </visual>
+    <collision>
+      <origin xyz="1.8748 -0.2935 0.075" rpy="-3.14159 1.54112e-16 -1.5708"/>
+      <geometry>
+        <mesh filename="file:///home/jay/ros2_ws/src/avone/description/assets/front_suspension.stl"/>
+      </geometry>
+    </collision>
+  <!-- REAR WHEEL HUB LEFT -->
+    <visual>
+      <origin xyz="-0.181377 0.297001 -0.105" rpy="6.30462e-15 0 -6.18615e-05"/>
+      <geometry>
+        <mesh filename="file:///home/jay/ros2_ws/src/avone/description/assets/rear_wheel_hub.stl"/>
+      </geometry>
+      <material name="white"/>
+    </visual>
+    <collision>
+      <origin xyz="-0.181377 0.297001 -0.105" rpy="6.30462e-15 0 -6.18615e-05"/>
+      <geometry>
+        <mesh filename="file:///home/jay/ros2_ws/src/avone/description/assets/rear_wheel_hub.stl"/>
+      </geometry>
+    </collision>
+  <!-- REAR WHEEL HUB RIGHT -->
     <visual>
       <origin xyz="0.181423 -0.296978 -0.105" rpy="3.10966e-15 7.00787e-15 -3.14153"/>
       <geometry>
-        <mesh filename="package://avone/avonemodel/assets/rear_wheel_hub.stl"/>
-      </geometry>
-      <material name="rear_wheel_hub_2_material">
-        <color rgba="0.972549 0.529412 0.00392157 1.0"/>
-      </material>
+        <mesh filename="file:///home/jay/ros2_ws/src/avone/description/assets/rear_wheel_hub.stl"/>
+      </geometry>
+      <material name="white"/>
     </visual>
     <collision>
       <origin xyz="0.181423 -0.296978 -0.105" rpy="3.10966e-15 7.00787e-15 -3.14153"/>
       <geometry>
-        <mesh filename="package://avone/avonemodel/assets/rear_wheel_hub.stl"/>
-      </geometry>
-    </collision>
-    <!-- Part rear_suspension -->
-    <visual>
-      <origin xyz="-0.17247 -0.28192 0.105" rpy="3.14159 5.47382e-48 -0.0851102"/>
-      <geometry>
-        <mesh filename="package://avone/avonemodel/assets/rear_suspension.stl"/>
-      </geometry>
-      <material name="rear_suspension_material">
-        <color rgba="0.647059 0.647059 0.647059 1.0"/>
-      </material>
-    </visual>
-    <collision>
-      <origin xyz="-0.17247 -0.28192 0.105" rpy="3.14159 5.47382e-48 -0.0851102"/>
-      <geometry>
-        <mesh filename="package://avone/avonemodel/assets/rear_suspension.stl"/>
-      </geometry>
-    </collision>
-    <!-- Part rear_suspension_2 -->
-    <visual>
-      <origin xyz="0.189017 0.312761 0.105" rpy="-3.14159 2.33363e-61 -3.05648"/>
-      <geometry>
-        <mesh filename="package://avone/avonemodel/assets/rear_suspension.stl"/>
-      </geometry>
-      <material name="rear_suspension_2_material">
-        <color rgba="0.647059 0.647059 0.647059 1.0"/>
-      </material>
-    </visual>
-    <collision>
-      <origin xyz="0.189017 0.312761 0.105" rpy="-3.14159 2.33363e-61 -3.05648"/>
-      <geometry>
-        <mesh filename="package://avone/avonemodel/assets/rear_suspension.stl"/>
-      </geometry>
-    </collision>
-    <!-- Part chassis -->
-    <visual>
-      <origin xyz="2.2924 -0.00985747 0.0751" rpy="3.14159 -0 1.5708"/>
-      <geometry>
-        <mesh filename="package://avone/avonemodel/assets/chassis.stl"/>
-      </geometry>
-      <material name="chassis_material">
-        <color rgba="0.615686 0.811765 0.929412 1.0"/>
-      </material>
-    </visual>
-    <collision>
-      <origin xyz="2.2924 -0.00985747 0.0751" rpy="3.14159 -0 1.5708"/>
-      <geometry>
-        <mesh filename="package://avone/avonemodel/assets/chassis.stl"/>
-      </geometry>
-    </collision>
-    <!-- Part front_suspension -->
-    <visual>
-      <origin xyz="2.0208 0.2935 0.075" rpy="3.14159 -1.54112e-16 1.5708"/>
-      <geometry>
-        <mesh filename="package://avone/avonemodel/assets/front_suspension.stl"/>
-      </geometry>
-      <material name="front_suspension_material">
-        <color rgba="0.231373 0.380392 0.705882 1.0"/>
-      </material>
-    </visual>
-    <collision>
-      <origin xyz="2.0208 0.2935 0.075" rpy="3.14159 -1.54112e-16 1.5708"/>
-      <geometry>
-        <mesh filename="package://avone/avonemodel/assets/front_suspension.stl"/>
-      </geometry>
-    </collision>
-    <!-- Part front_suspension_2 -->
-    <visual>
-      <origin xyz="2.2924 -0.2935 0.075" rpy="-3.14159 1.54112e-16 -1.5708"/>
-      <geometry>
-        <mesh filename="package://avone/avonemodel/assets/front_suspension.stl"/>
-      </geometry>
-      <material name="front_suspension_2_material">
-        <color rgba="0.231373 0.380392 0.705882 1.0"/>
-      </material>
-    </visual>
-    <collision>
-      <origin xyz="2.2924 -0.2935 0.075" rpy="-3.14159 1.54112e-16 -1.5708"/>
-      <geometry>
-        <mesh filename="package://avone/avonemodel/assets/front_suspension.stl"/>
+        <mesh filename="file:///home/jay/ros2_ws/src/avone/description/assets/rear_wheel_hub.stl"/>
       </geometry>
     </collision>
   </link>
-  <!-- Link wheel -->
-  <link name="wheel">
-    <inertial>
-      <origin xyz="-8.09407e-17 -1.33567e-17 0.0496398" rpy="0 0 0"/>
-      <mass value="9.8"/>
-      <inertia ixx="0.169474" ixy="2.12205e-15" ixz="6.60536e-16" iyy="0.169474" iyz="1.10915e-15" izz="0.253875"/>
-    </inertial>
-    <!-- Part wheel -->
-    <visual>
-      <origin xyz="-8.09391e-17 7.65875e-18 0.17" rpy="1.5708 -3.89756e-15 3.70519e-15"/>
-      <geometry>
-        <mesh filename="package://avone/avonemodel/assets/wheel.stl"/>
-      </geometry>
-      <material name="wheel_material">
-        <color rgba="0.917647 0.917647 0.917647 1.0"/>
-      </material>
-    </visual>
-    <collision>
-      <origin xyz="-8.09391e-17 7.65875e-18 0.17" rpy="1.5708 -3.89756e-15 3.70519e-15"/>
-      <geometry>
-        <mesh filename="package://avone/avonemodel/assets/wheel.stl"/>
-      </geometry>
-    </collision>
-  </link>
-  <!-- Joint from chassis_suspension to wheel -->
-  <joint name="RLMotor" type="revolute">
-    <origin xyz="4.71381e-05 0.693977 3.30291e-15" rpy="1.5708 -0 -6.18615e-05"/>
-    <parent link="chassis_suspension"/>
-    <child link="wheel"/>
-    <axis xyz="0 0 1"/>
-    <limit effort="10" velocity="10" lower="-3.141592653589793" upper="3.141592653589793"/>
-  </joint>
-  <!-- Link wheel_2 -->
-  <link name="wheel_2">
-    <inertial>
-      <origin xyz="-1.66794e-17 -1.33614e-17 0.0496398" rpy="0 0 0"/>
-      <mass value="9.8"/>
-      <inertia ixx="0.169474" ixy="1.1918e-15" ixz="-3.1455e-16" iyy="0.169474" iyz="5.0174e-16" izz="0.253875"/>
-    </inertial>
-    <!-- Part wheel_2 -->
-    <visual>
-      <origin xyz="-1.59877e-17 7.65404e-18 0.17" rpy="1.5708 1.86465e-15 -5.13481e-16"/>
-      <geometry>
-        <mesh filename="package://avone/avonemodel/assets/wheel.stl"/>
-      </geometry>
-      <material name="wheel_2_material">
-        <color rgba="0.917647 0.917647 0.917647 1.0"/>
-      </material>
-    </visual>
-    <collision>
-      <origin xyz="-1.59877e-17 7.65404e-18 0.17" rpy="1.5708 1.86465e-15 -5.13481e-16"/>
-      <geometry>
-        <mesh filename="package://avone/avonemodel/assets/wheel.stl"/>
-      </geometry>
-    </collision>
-  </link>
-  <!-- Joint from chassis_suspension to wheel_2 -->
-  <joint name="RRMotor" type="revolute">
-    <origin xyz="4.71381e-05 -0.693977 2.30371e-15" rpy="1.5708 7.00787e-15 -3.14153"/>
-    <parent link="chassis_suspension"/>
-    <child link="wheel_2"/>
-    <axis xyz="0 0 1"/>
-    <limit effort="10" velocity="10" lower="-3.141592653589793" upper="3.141592653589793"/>
-  </joint>
-  <!-- Link front_wheel_hub -->
-  <link name="front_wheel_hub">
-    <inertial>
-      <origin xyz="0.0824722 -5.82867e-16 0.09" rpy="0 0 0"/>
-      <mass value="1.6"/>
-      <inertia ixx="0.00734348" ixy="-1.63364e-18" ixz="-3.73248e-19" iyy="0.00420677" iyz="6.09249e-20" izz="0.00395986"/>
-    </inertial>
-    <!-- Part front_wheel_hub -->
-    <visual>
-      <origin xyz="-0.290639 0.1358 0.18" rpy="-3.14159 1.1031e-16 -5.55112e-17"/>
-      <geometry>
-        <mesh filename="package://avone/avonemodel/assets/front_wheel_hub.stl"/>
-      </geometry>
-      <material name="front_wheel_hub_material">
-        <color rgba="0.768627 0.886275 0.952941 1.0"/>
-      </material>
-    </visual>
-    <collision>
-      <origin xyz="-0.290639 0.1358 0.18" rpy="-3.14159 1.1031e-16 -5.55112e-17"/>
-      <geometry>
-        <mesh filename="package://avone/avonemodel/assets/front_wheel_hub.stl"/>
-      </geometry>
-    </collision>
-  </link>
-  <!-- Link wheel_3 -->
-  <link name="wheel_3">
-    <inertial>
-      <origin xyz="1.09934e-17 -1.19492e-32 0.0496398" rpy="0 0 0"/>
-      <mass value="9.8"/>
-      <inertia ixx="0.169474" ixy="1.82963e-33" ixz="4.67592e-18" iyy="0.169474" iyz="9.43037e-33" izz="0.253875"/>
-    </inertial>
-    <!-- Part wheel_3 -->
-    <visual>
-      <origin xyz="0 0 0.17" rpy="1.5708 9.24446e-32 1.5708"/>
-      <geometry>
-        <mesh filename="package://avone/avonemodel/assets/wheel.stl"/>
-      </geometry>
-      <material name="wheel_3_material">
-        <color rgba="0.917647 0.917647 0.917647 1.0"/>
-      </material>
-    </visual>
-    <collision>
-      <origin xyz="0 0 0.17" rpy="1.5708 9.24446e-32 1.5708"/>
-      <geometry>
-        <mesh filename="package://avone/avonemodel/assets/wheel.stl"/>
-      </geometry>
-    </collision>
-  </link>
-  <!-- Joint from front_wheel_hub to wheel_3 -->
-  <joint name="FRwheel" type="revolute">
-    <origin xyz="0.10836 -4.44089e-16 0.09" rpy="1.5708 2.46751e-16 -1.5708"/>
-    <parent link="front_wheel_hub"/>
-    <child link="wheel_3"/>
-    <axis xyz="0 0 1"/>
-    <limit effort="10" velocity="10" lower="-3.141592653589793" upper="3.141592653589793"/>
-  </joint>
-  <!-- Joint from chassis_suspension to front_wheel_hub -->
-  <joint name="RSteer" type="revolute">
-    <origin xyz="2.1566 -0.584139 0.075" rpy="-3.14159 1.54112e-16 -1.5708"/>
-    <parent link="chassis_suspension"/>
-    <child link="front_wheel_hub"/>
-    <axis xyz="0 0 1"/>
-    <limit effort="10" velocity="10" lower="-3.141592653589793" upper="3.141592653589793"/>
-  </joint>
-  <!-- Link front_wheel_hub_2 -->
-  <link name="front_wheel_hub_2">
-    <inertial>
-      <origin xyz="0.0824722 -7.49401e-16 0.09" rpy="0 0 0"/>
-      <mass value="1.6"/>
-      <inertia ixx="0.00734348" ixy="-4.21008e-17" ixz="3.73248e-19" iyy="0.00420677" iyz="-6.18738e-20" izz="0.00395986"/>
-    </inertial>
-    <!-- Part front_wheel_hub_2 -->
-    <visual>
-      <origin xyz="-0.290639 0.1358 0.18" rpy="3.14159 -1.1031e-16 -1.385e-14"/>
-      <geometry>
-        <mesh filename="package://avone/avonemodel/assets/front_wheel_hub.stl"/>
-      </geometry>
-      <material name="front_wheel_hub_2_material">
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