Commit message: re-organise of code before first autonomous drive, creation of sectioned launch files

File: src/avone/description/robot.urdf.xacro (robot description, xacro)
@@ -3,5 +3,7 @@
   <!-- 2) Core links/visuals etc -->
   <xacro:include filename="robot_core.xacro"/>
+  <!-- FOR SIMULATION -->
   <!-- <xacro:include filename="ros2_control.xacro"/> -->
+  <!-- FOR REAL HARDWARE -->
   <xacro:include filename="ros2_control_hardware.xacro"/>
   <!-- 5) Sensors, cameras, lidar, etc. -->

File: src/avone/description/robot_core.xacro (robot description, xacro)
@@ -3,5 +3,5 @@
     <xacro:include filename="inertial_macros.xacro"/>
     <!-- change this to local directroy -->
-    <!-- <xacro:arg name="mesh_dir" default="file://home/avone/avone_ws/src/avone/description/assets"/> -->
+    <!-- <xacro:arg name="mesh_dir" default="file://home/jay/ros2_ws/src/avone/description/assets"/> -->
     <material name="white">
         <color rgba="1 1 1 1" />
@@ -38,6 +38,6 @@
             <origin xyz="2.2924 -0.00985747 0.0751" rpy="3.14159 0 1.5708"/>
             <geometry>
-                  <!-- <mesh filename="file:///home/avone/avone_ws/src/avone/description/assets/chassis.stl"/> -->
-                  <mesh filename="file:///home/avone/avone_ws/src/avone/description/assets/chassis.stl"/>
+                  <!-- <mesh filename="file:///home/jay/ros2_ws/src/avone/description/assets/chassis.stl"/> -->
+                  <mesh filename="file:///home/jay/ros2_ws/src/avone/description/assets/chassis.stl"/>
 <!-- home/jay/ros2_ws/src/avone -->
                  <!--  <box size="0.3 0.3 0.15"/> -->
@@ -48,5 +48,5 @@
             <origin xyz="2.2924 -0.00985747 0.0751" rpy="3.14159 0 1.5708"/>
             <geometry>
-                    <mesh filename="file:///home/avone/avone_ws/src/avone/description/assets/chassis.stl"/>
+                    <mesh filename="file:///home/jay/ros2_ws/src/avone/description/assets/chassis.stl"/>
                  <!--  <box size="0.3 0.3 0.15"/> -->
             </geometry>
@@ -59,5 +59,5 @@
       <origin xyz="-0.170629 -0.28192 0.105" rpy="3.14159 5.47382e-48 -0.0851102"/>
       <geometry>
-        <mesh filename="file:///home/avone/avone_ws/src/avone/description/assets/rear_suspension.stl"/>
+        <mesh filename="file:///home/jay/ros2_ws/src/avone/description/assets/rear_suspension.stl"/>
       </geometry>
       <material name="blue"/>
@@ -66,5 +66,5 @@
       <origin xyz="-0.170629 -0.28192 0.105" rpy="3.14159 5.47382e-48 -0.0851102"/>
       <geometry>
-        <mesh filename="file:///home/avone/avone_ws/src/avone/description/assets/rear_suspension.stl"/>
+        <mesh filename="file:///home/jay/ros2_ws/src/avone/description/assets/rear_suspension.stl"/>
       </geometry>
     </collision>
@@ -73,5 +73,5 @@
       <origin xyz="0.189017 0.312761 0.105" rpy="-3.14159 2.33363e-61 -3.05648"/>
       <geometry>
-        <mesh filename="file:///home/avone/avone_ws/src/avone/description/assets/rear_suspension.stl"/>
+        <mesh filename="file:///home/jay/ros2_ws/src/avone/description/assets/rear_suspension.stl"/>
       </geometry>
       <material name="blue"/>
@@ -80,5 +80,5 @@
       <origin xyz="0.189017 0.312761 0.105" rpy="-3.14159 2.33363e-61 -3.05648"/>
       <geometry>
-        <mesh filename="file:///home/avone/avone_ws/src/avone/description/assets/rear_suspension.stl"/>
+        <mesh filename="file:///home/jay/ros2_ws/src/avone/description/assets/rear_suspension.stl"/>
       </geometry>
     </collision>
@@ -87,5 +87,5 @@
       <origin xyz="1.6032 0.2935 0.075" rpy="3.14159 -1.54112e-16 1.5708"/>
       <geometry>
-        <mesh filename="file:///home/avone/avone_ws/src/avone/description/assets/front_suspension.stl"/>
+        <mesh filename="file:///home/jay/ros2_ws/src/avone/description/assets/front_suspension.stl"/>
       </geometry>
       <material name="blue"/>
@@ -94,5 +94,5 @@
       <origin xyz="1.6032 0.2935 0.075" rpy="3.14159 -1.54112e-16 1.5708"/>
       <geometry>
-        <mesh filename="file:///home/avone/avone_ws/src/avone/description/assets/front_suspension.stl"/>
+        <mesh filename="file:///home/jay/ros2_ws/src/avone/description/assets/front_suspension.stl"/>
       </geometry>
     </collision>
@@ -101,5 +101,5 @@
       <origin xyz="1.8748 -0.2935 0.075" rpy="-3.14159 1.54112e-16 -1.5708"/>
       <geometry>
-        <mesh filename="file:///home/avone/avone_ws/src/avone/description/assets/front_suspension.stl"/>
+        <mesh filename="file:///home/jay/ros2_ws/src/avone/description/assets/front_suspension.stl"/>
       </geometry>
       <material name="blue"/>
@@ -108,5 +108,5 @@
       <origin xyz="1.8748 -0.2935 0.075" rpy="-3.14159 1.54112e-16 -1.5708"/>
       <geometry>
-        <mesh filename="file:///home/avone/avone_ws/src/avone/description/assets/front_suspension.stl"/>
+        <mesh filename="file:///home/jay/ros2_ws/src/avone/description/assets/front_suspension.stl"/>
       </geometry>
     </collision>
@@ -115,5 +115,5 @@
       <origin xyz="-0.181377 0.297001 -0.105" rpy="6.30462e-15 0 -6.18615e-05"/>
       <geometry>
-        <mesh filename="file:///home/avone/avone_ws/src/avone/description/assets/rear_wheel_hub.stl"/>
+        <mesh filename="file:///home/jay/ros2_ws/src/avone/description/assets/rear_wheel_hub.stl"/>
       </geometry>
       <material name="white"/>
@@ -122,5 +122,5 @@
       <origin xyz="-0.181377 0.297001 -0.105" rpy="6.30462e-15 0 -6.18615e-05"/>
       <geometry>
-        <mesh filename="file:///home/avone/avone_ws/src/avone/description/assets/rear_wheel_hub.stl"/>
+        <mesh filename="file:///home/jay/ros2_ws/src/avone/description/assets/rear_wheel_hub.stl"/>
       </geometry>
     </collision>
@@ -129,5 +129,5 @@
       <origin xyz="0.181423 -0.296978 -0.105" rpy="3.10966e-15 7.00787e-15 -3.14153"/>
       <geometry>
-        <mesh filename="file:///home/avone/avone_ws/src/avone/description/assets/rear_wheel_hub.stl"/>
+        <mesh filename="file:///home/jay/ros2_ws/src/avone/description/assets/rear_wheel_hub.stl"/>
       </geometry>
       <material name="white"/>
@@ -136,5 +136,5 @@
       <origin xyz="0.181423 -0.296978 -0.105" rpy="3.10966e-15 7.00787e-15 -3.14153"/>
       <geometry>
-        <mesh filename="file:///home/avone/avone_ws/src/avone/description/assets/rear_wheel_hub.stl"/>
+        <mesh filename="file:///home/jay/ros2_ws/src/avone/description/assets/rear_wheel_hub.stl"/>
       </geometry>
     </collision>
@@ -166,5 +166,5 @@
             <origin xyz="-8.09391e-17 7.65875e-18 0.17" rpy="1.5708 0 0"/>
             <geometry>
-                    <mesh filename="file:///home/avone/avone_ws/src/avone/description/assets/wheel.stl"/>
+                    <mesh filename="file:///home/jay/ros2_ws/src/avone/description/assets/wheel.stl"/>
                  <!--  <box size="0.3 0.3 0.15"/> -->
             </geometry>
@@ -174,5 +174,5 @@
             <origin xyz="-8.09391e-17 7.65875e-18 0.17" rpy="1.5708 0 0"/>
             <geometry>
-                     <!--<mesh filename="file:///home/avone/avone_ws/src/avone/description/assets/wheel.stl"/>    -->
+                     <!--<mesh filename="file:///home/jay/ros2_ws/src/avone/description/assets/wheel.stl"/>    -->
                                         <sphere radius="0.203"/>
                  <!--  <box size="0.3 0.3 0.15"/> -->
@@ -201,5 +201,5 @@
             <origin xyz="-1.59877e-17 7.65404e-18 0.17" rpy="1.5708 0 0"/>
             <geometry>
-                    <mesh filename="file:///home/avone/avone_ws/src/avone/description/assets/wheel.stl"/>
+                    <mesh filename="file:///home/jay/ros2_ws/src/avone/description/assets/wheel.stl"/>
                  <!--  <box size="0.3 0.3 0.15"/> -->
             </geometry>
@@ -237,5 +237,5 @@
             <origin xyz="-0.290639 0.1358 0.18" rpy="-3.14159 0 0"/>
             <geometry>
-                    <mesh filename="file:///home/avone/avone_ws/src/avone/description/assets/front_wheel_hub.stl"/>
+                    <mesh filename="file:///home/jay/ros2_ws/src/avone/description/assets/front_wheel_hub.stl"/>
                  <!--  <box size="0.3 0.3 0.15"/> -->
             </geometry>
@@ -245,5 +245,5 @@
             <origin xyz="-0.290639 0.1358 0.18" rpy="-3.14159 0 0"/>
             <geometry>
-                    <mesh filename="file:///home/avone/avone_ws/src/avone/description/assets/front_wheel_hub.stl"/>
+                    <mesh filename="file:///home/jay/ros2_ws/src/avone/description/assets/front_wheel_hub.stl"/>
                  <!--  <box size="0.3 0.3 0.15"/> -->
             </geometry>
@@ -268,5 +268,5 @@
             <origin xyz="2.22045e-16 0 0.17" rpy="1.5708 0 1.5708"/>
             <geometry>
-                    <mesh filename="file:///home/avone/avone_ws/src/avone/description/assets/wheel.stl"/>
+                    <mesh filename="file:///home/jay/ros2_ws/src/avone/description/assets/wheel.stl"/>
                  <!--  <box size="0.3 0.3 0.15"/> -->
             </geometry>
@@ -276,5 +276,5 @@
             <origin xyz="2.22045e-16 0 0.17" rpy="1.5708 0 1.5708"/>
             <geometry>
-                   <!--<mesh filename="file:///home/avone/avone_ws/src/avone/description/assets/wheel.stl"/>    -->
+                   <!--<mesh filename="file:///home/jay/ros2_ws/src/avone/description/assets/wheel.stl"/>    -->
                                         <sphere radius="0.203"/>
                  <!--  <box size="0.3 0.3 0.15"/> -->
@@ -304,5 +304,5 @@
         <origin xyz="-0.290639 0.1358 0.18" rpy="3.14159 0 0"/>
         <geometry>
-                    <mesh filename="file:///home/avone/avone_ws/src/avone/description/assets/front_wheel_hub.stl"/>
+                    <mesh filename="file:///home/jay/ros2_ws/src/avone/description/assets/front_wheel_hub.stl"/>
                  <!--  <box size="0.3 0.3 0.15"/> -->
         </geometry>
@@ -312,5 +312,5 @@
         <origin xyz="-0.290639 0.1358 0.18" rpy="3.14159 0 0"/>
         <geometry>
-                    <mesh filename="file:///home/avone/avone_ws/src/avone/description/assets/front_wheel_hub.stl"/>
+                    <mesh filename="file:///home/jay/ros2_ws/src/avone/description/assets/front_wheel_hub.stl"/>
                  <!--  <box size="0.3 0.3 0.15"/> -->
         </geometry>
@@ -335,5 +335,5 @@
         <origin xyz="0 0 0.17" rpy="1.5708 0 0"/>
         <geometry>
-                    <mesh filename="file:///home/avone/avone_ws/src/avone/description/assets/wheel.stl"/>
+                    <mesh filename="file:///home/jay/ros2_ws/src/avone/description/assets/wheel.stl"/>
                  <!--  <box size="0.3 0.3 0.15"/> -->
         </geometry>
@@ -343,5 +343,5 @@
         <origin xyz="0 0 0.17" rpy="1.5708 0 0"/>
         <geometry>
-                      <!--<mesh filename="file:///home/avone/avone_ws/src/avone/description/assets/wheel.stl"/>    -->
+                      <!--<mesh filename="file:///home/jay/ros2_ws/src/avone/description/assets/wheel.stl"/>    -->
                                         <sphere radius="0.203"/>
                  <!--  <box size="0.3 0.3 0.15"/> -->

File: src/avone/description/ros2_control_hardware.xacro (robot description, xacro)
@@ -5,6 +5,6 @@
       <plugin>avone/AvoneSystemHardware</plugin>
       <!-- Your existing params -->
-      <param name="max_steer_angle">1.3</param>
-      <param name="min_steer_angle">-1.3</param>
+      <param name="max_steer_angle">0.610865</param>
+      <param name="min_steer_angle">-0.610865</param>
       <param name="max_rpm">350</param>
       <param name="can_interface">can0</param>
@@ -17,26 +17,4 @@
       <param name="cmd_r_motor_can_id">0x0A</param>
       <param name="cmd_steer_can_id">0x09</param>
-      <!-- NEW: safety/watchdog controls -->
-      <!-- Which feedback signals are required before arming & during run -->
-      <param name="require_rlmotor">false</param>
-      <param name="require_rrmotor">false</param>
-      <param name="require_steer">false</param>
-      <!-- Activation: wait up to this long for first feedback frames -->
-      <param name="startup_validation_ms">800</param>
-      <!-- Runtime: max allowed age for any required signal -->
-      <param name="link_loss_timeout_ms">250</param>
-            <!-- LiDAR watchdog -->
-      <param name="require_lidar">false</param>
-      <param name="lidar_topic">/lidar</param>
-      <!-- Choose the actual ROS 2 type your stack publishes: -->
-      <param name="lidar_ros_type">sensor_msgs/msg/PointCloud2</param>
-      <!-- or -->
-      <!-- <param name="lidar_ros_type">sensor_msgs/msg/LaserScan</param> -->
-      <param name="lidar_timeout_ms">300</param>
-      <!-- Ready-To-Drive signalling -->
-      <param name="r2d_topic">/ready_to_drive</param>
-      <param name="r2d_can_heartbeat">true</param>
-      <param name="r2d_can_id">0x110</param>
-      <param name="r2d_can_period_ms">50</param>
     </hardware>
     <!-- front steering -->

File: src/avone/description/sensors.xacro (robot description, xacro)
@@ -17,10 +17,10 @@
   </gazebo>
   <!-- FRONT GPS ANTENNA -->
-  <joint name="gps_antenna1_joint" type="fixed">
+  <joint name="gps_joint" type="fixed">
         <parent link="chassis"/>
-        <child link="gps_antenna1_link"/>
+        <child link="gps_link"/>
           <origin xyz="0.0312 0 0.3924" rpy="0 0 0"/>
     </joint>
-  <link name="gps_antenna1_link">
+  <link name="gps_link">
     <visual>
       <geometry>
@@ -35,7 +35,7 @@
     </collision>
   </link>
-  <gazebo reference="gps_antenna1_link">
+  <gazebo reference="gps_link">
     <sensor name="navsat1" type="navsat">
-    <gz_frame_id>gps_antenna1_link</gz_frame_id>
+    <gz_frame_id>gps_link</gz_frame_id>
       <always_on>1</always_on>
       <update_rate>50</update_rate>

Commit message: updated drive and localisation programs after first autonomous drive

File: src/avone/description/robot.urdf.xacro (robot description, xacro)
@@ -4,7 +4,7 @@
   <xacro:include filename="robot_core.xacro"/>
   <!-- FOR SIMULATION -->
-  <xacro:include filename="ros2_control.xacro"/>
+  <!-- <xacro:include filename="ros2_control.xacro"/> -->
   <!-- FOR REAL HARDWARE -->
-  <!-- <xacro:include filename="ros2_control_hardware.xacro"/> -->
+  <xacro:include filename="ros2_control_hardware.xacro"/>
   <!-- 5) Sensors, cameras, lidar, etc. -->
   <xacro:include filename="camera.xacro"/>

File: src/avone/description/sensors.xacro (robot description, xacro)
@@ -17,10 +17,10 @@
   </gazebo>
   <!-- FRONT GPS ANTENNA -->
-  <joint name="gps_joint" type="fixed">
+  <joint name="gps_joint1" type="fixed">
         <parent link="chassis"/>
-        <child link="gps_link"/>
-          <origin xyz="0.0312 0 0.3924" rpy="0 0 0"/>
+        <child link="gps_link1"/>
+          <origin xyz="-0.1188 0 0.3924" rpy="0 0 0"/>
     </joint>
-  <link name="gps_link">
+  <link name="gps_link1">
     <visual>
       <geometry>
@@ -35,7 +35,7 @@
     </collision>
   </link>
-  <gazebo reference="gps_link">
+  <gazebo reference="gps_link1">
     <sensor name="navsat1" type="navsat">
-    <gz_frame_id>gps_link</gz_frame_id>
+    <gz_frame_id>gps_link1</gz_frame_id>
       <always_on>1</always_on>
       <update_rate>50</update_rate>
@@ -47,10 +47,10 @@
     </sensor>
   </gazebo>
-<joint name="gps_antenna2_joint" type="fixed">
+<joint name="gps_joint2" type="fixed">
         <parent link="chassis"/>
-        <child link="gps_antenna2_link"/>
+        <child link="gps_link2"/>
           <origin xyz="2.131 0 0.3924" rpy="0 0 0"/>
     </joint>
-  <link name="gps_antenna2_link">
+  <link name="gps_link2">
    <visual>
       <geometry>
@@ -65,7 +65,7 @@
     </collision>
   </link>
-  <gazebo reference="gps_antenna2_link">
+  <gazebo reference="gps_link2">
     <sensor name="navsat2" type="navsat">
-    <gz_frame_id>gps_antenna2_link</gz_frame_id>
+    <gz_frame_id>gps_link2</gz_frame_id>
       <always_on>1</always_on>
       <update_rate>50</update_rate>
