Commit message: Final commit to avone ros2 workspace from father, cleaning and preparing to move on, as a tear drops down my cheek, and a white monster down my gut, i will forever love you my child

File: src/avone/description/robot.urdf.xacro (robot description, xacro)
@@ -9,7 +9,7 @@
   <!-- Control interface -->
   <!-- FOR SIMULATION -->
-  <xacro:include filename="ros2_control.xacro"/>
+  <!-- <xacro:include filename="ros2_control.xacro"/> -->
   <!-- FOR REAL HARDWARE -->
-  <!-- <xacro:include filename="ros2_control_hardware.xacro"/> -->
+  <xacro:include filename="ros2_control_hardware.xacro"/>
  <!-- Sensors, cameras, lidar, etc. -->
   <xacro:include filename="camera.xacro"/>

File: src/avone/description/robot_core.xacro (robot description, xacro)
@@ -76,5 +76,5 @@
       <origin xyz="2.2924 -0.00985747 0.0751" rpy="3.14159 0 1.5708"/>
       <geometry>
-        <mesh filename="file:///home/avone/avone_ws/src/avone/description/assets/chassis.stl"/>
+        <mesh filename="package://avone/description/assets/chassis.stl"/>
       </geometry>
       <material name="blue"/>
@@ -83,5 +83,5 @@
       <origin xyz="2.2924 -0.00985747 0.0751" rpy="3.14159 0 1.5708"/>
       <geometry>
-        <mesh filename="file:///home/avone/avone_ws/src/avone/description/assets/chassis.stl"/>
+        <mesh filename="package://avone/description/assets/chassis.stl"/>
       </geometry>
     </collision>
@@ -97,5 +97,5 @@
       <origin xyz="-0.170629 -0.28192 0.105" rpy="3.14159 5.47382e-48 -0.0851102"/>
       <geometry>
-        <mesh filename="file:///home/avone/avone_ws/src/avone/description/assets/rear_suspension.stl"/>
+        <mesh filename="package://avone/description/assets/rear_suspension.stl"/>
       </geometry>
       <material name="blue"/>
@@ -104,5 +104,5 @@
       <origin xyz="-0.170629 -0.28192 0.105" rpy="3.14159 5.47382e-48 -0.0851102"/>
       <geometry>
-        <mesh filename="file:///home/avone/avone_ws/src/avone/description/assets/rear_suspension.stl"/>
+        <mesh filename="package://avone/description/assets/rear_suspension.stl"/>
       </geometry>
     </collision>
@@ -111,5 +111,5 @@
       <origin xyz="0.189017 0.312761 0.105" rpy="-3.14159 2.33363e-61 -3.05648"/>
       <geometry>
-        <mesh filename="file:///home/avone/avone_ws/src/avone/description/assets/rear_suspension.stl"/>
+        <mesh filename="package://avone/description/assets/rear_suspension.stl"/>
       </geometry>
       <material name="blue"/>
@@ -118,5 +118,5 @@
       <origin xyz="0.189017 0.312761 0.105" rpy="-3.14159 2.33363e-61 -3.05648"/>
       <geometry>
-        <mesh filename="file:///home/avone/avone_ws/src/avone/description/assets/rear_suspension.stl"/>
+        <mesh filename="package://avone/description/assets/rear_suspension.stl"/>
       </geometry>
     </collision>
@@ -128,5 +128,5 @@
       <origin xyz="1.6032 0.2935 0.075" rpy="3.14159 -1.54112e-16 1.5708"/>
       <geometry>
-        <mesh filename="file:///home/avone/avone_ws/src/avone/description/assets/front_suspension.stl"/>
+        <mesh filename="package://avone/description/assets/front_suspension.stl"/>
       </geometry>
       <material name="blue"/>
@@ -135,5 +135,5 @@
       <origin xyz="1.6032 0.2935 0.075" rpy="3.14159 -1.54112e-16 1.5708"/>
       <geometry>
-        <mesh filename="file:///home/avone/avone_ws/src/avone/description/assets/front_suspension.stl"/>
+        <mesh filename="package://avone/description/assets/front_suspension.stl"/>
       </geometry>
     </collision>
@@ -142,5 +142,5 @@
       <origin xyz="1.8748 -0.2935 0.075" rpy="-3.14159 1.54112e-16 -1.5708"/>
       <geometry>
-        <mesh filename="file:///home/avone/avone_ws/src/avone/description/assets/front_suspension.stl"/>
+        <mesh filename="package://avone/description/assets/front_suspension.stl"/>
       </geometry>
       <material name="blue"/>
@@ -149,5 +149,5 @@
       <origin xyz="1.8748 -0.2935 0.075" rpy="-3.14159 1.54112e-16 -1.5708"/>
       <geometry>
-        <mesh filename="file:///home/avone/avone_ws/src/avone/description/assets/front_suspension.stl"/>
+        <mesh filename="package://avone/description/assets/front_suspension.stl"/>
       </geometry>
     </collision>
@@ -159,5 +159,5 @@
       <origin xyz="-0.181377 0.297001 -0.105" rpy="6.30462e-15 0 -6.18615e-05"/>
       <geometry>
-        <mesh filename="file:///home/avone/avone_ws/src/avone/description/assets/rear_wheel_hub.stl"/>
+        <mesh filename="package://avone/description/assets/rear_wheel_hub.stl"/>
       </geometry>
       <material name="white"/>
@@ -166,5 +166,5 @@
       <origin xyz="-0.181377 0.297001 -0.105" rpy="6.30462e-15 0 -6.18615e-05"/>
       <geometry>
-        <mesh filename="file:///home/avone/avone_ws/src/avone/description/assets/rear_wheel_hub.stl"/>
+        <mesh filename="package://avone/description/assets/rear_wheel_hub.stl"/>
       </geometry>
     </collision>
@@ -173,5 +173,5 @@
       <origin xyz="0.181423 -0.296978 -0.105" rpy="3.10966e-15 7.00787e-15 -3.14153"/>
       <geometry>
-        <mesh filename="file:///home/avone/avone_ws/src/avone/description/assets/rear_wheel_hub.stl"/>
+        <mesh filename="package://avone/description/assets/rear_wheel_hub.stl"/>
       </geometry>
       <material name="white"/>
@@ -180,5 +180,5 @@
       <origin xyz="0.181423 -0.296978 -0.105" rpy="3.10966e-15 7.00787e-15 -3.14153"/>
       <geometry>
-        <mesh filename="file:///home/avone/avone_ws/src/avone/description/assets/rear_wheel_hub.stl"/>
+        <mesh filename="package://avone/description/assets/rear_wheel_hub.stl"/>
       </geometry>
     </collision>
@@ -206,5 +206,5 @@
       <origin xyz="-8.09391e-17 7.65875e-18 0.17" rpy="1.5708 0 0"/>
       <geometry>
-        <mesh filename="file:///home/avone/avone_ws/src/avone/description/assets/wheel.stl"/>
+        <mesh filename="package://avone/description/assets/wheel.stl"/>
       </geometry>
       <material name="black"/>
@@ -237,5 +237,5 @@
       <origin xyz="-1.59877e-17 7.65404e-18 0.17" rpy="1.5708 0 0"/>
       <geometry>
-        <mesh filename="file:///home/avone/avone_ws/src/avone/description/assets/wheel.stl"/>
+        <mesh filename="package://avone/description/assets/wheel.stl"/>
       </geometry>
       <material name="black"/>
@@ -270,5 +270,5 @@
       <origin xyz="-0.290639 0.1358 0.18" rpy="-3.14159 0 0"/>
       <geometry>
-        <mesh filename="file:///home/avone/avone_ws/src/avone/description/assets/front_wheel_hub.stl"/>
+        <mesh filename="package://avone/description/assets/front_wheel_hub.stl"/>
       </geometry>
       <material name="white"/>
@@ -277,5 +277,5 @@
       <origin xyz="-0.290639 0.1358 0.18" rpy="-3.14159 0 0"/>
       <geometry>
-        <mesh filename="file:///home/avone/avone_ws/src/avone/description/assets/front_wheel_hub.stl"/>
+        <mesh filename="package://avone/description/assets/front_wheel_hub.stl"/>
       </geometry>
     </collision>
@@ -300,5 +300,5 @@
       <origin xyz="2.22045e-16 0 0.17" rpy="1.5708 0 1.5708"/>
       <geometry>
-        <mesh filename="file:///home/avone/avone_ws/src/avone/description/assets/wheel.stl"/>
+        <mesh filename="package://avone/description/assets/wheel.stl"/>
       </geometry>
       <material name="black"/>
@@ -333,5 +333,5 @@
       <origin xyz="-0.290639 0.1358 0.18" rpy="3.14159 0 0"/>
       <geometry>
-        <mesh filename="file:///home/avone/avone_ws/src/avone/description/assets/front_wheel_hub.stl"/>
+        <mesh filename="package://avone/description/assets/front_wheel_hub.stl"/>
       </geometry>
       <material name="white"/>
@@ -340,5 +340,5 @@
       <origin xyz="-0.290639 0.1358 0.18" rpy="3.14159 0 0"/>
       <geometry>
-        <mesh filename="file:///home/avone/avone_ws/src/avone/description/assets/front_wheel_hub.stl"/>
+        <mesh filename="package://avone/description/assets/front_wheel_hub.stl"/>
       </geometry>
     </collision>
@@ -363,5 +363,5 @@
       <origin xyz="0 0 0.17" rpy="1.5708 0 0"/>
       <geometry>
-        <mesh filename="file:///home/avone/avone_ws/src/avone/description/assets/wheel.stl"/>
+        <mesh filename="package://avone/description/assets/wheel.stl"/>
       </geometry>
       <material name="black"/>
